File: hardware/kicad/ver_1.0/MSBE_V3.kicad_pcb (KiCad board)
At the start: 4 copper layers, 145 parts, among them J1 USB_C_Receptacle_USB2.0_16P, J10 Low-V, J2 USB_C_Receptacle_USB2.0_16P, J3 Touch Pads, J4 Touch Pads, J5 UART, J6 UART, J7 Prog, J8 Prog, J9 High-V, U1 NPM1100-CAAA-R7, U10 MAX98357AEWL_T, U2 NPM1100-CAAA-R7, U3 NRF5340-CLAA-R, U4 NRF5340-CLAA-R, U5 BMA400, U6 BMA400, U7 MPR121QR2, U8 MPR121QR2, U9 MAX98357AEWL_T, Y1 Crystal, Y2 Crystal

Commit message: update
Parts:
- added AE1: Antenna_Shield, RF_Antenna:Texas_SWRA117D_2.4GHz_Left, F.Cu at (-104.2, 107.7)
- added AE2: Antenna_Shield, RF_Antenna:Texas_SWRA117D_2.4GHz_Left, F.Cu at (-104.2, 100.6)
- added C72: 100nF, Capacitor_SMD:C_0603_1608Metric, F.Cu at (-111.0, 93.1)
- added C73: 100nF, Capacitor_SMD:C_0603_1608Metric, F.Cu at (-107.0, 63.0)
- added C74: 100nF, Capacitor_SMD:C_0603_1608Metric, F.Cu at (-107.0, 65.5)
- added C75: 100nF, Capacitor_SMD:C_0603_1608Metric, F.Cu at (-107.0, 68.0)
- added J11: UART, myLib:Pad_3Pin_1.5x0.8mm, F.Cu at (-135.1, 35.6)
- added L10: 2.2uH, Inductor_SMD:L_0603_1608Metric, F.Cu at (-95.0, 90.6)
- added L9: 10uH, Inductor_SMD:L_0603_1608Metric, F.Cu at (-91.0, 63.0)
- added Y3: 32MHz, myLib:ECS-160-10-37-JTN-TR_ECS, F.Cu at (-125.1, 59.0)
- added Y4: 32.768kHz, myLib:Crystal_24MHz-ECS-240-12-37B-CKY-TR, F.Cu at (-126.4, 42.8)
- BT1, BT2: footprint myLib:Pad_2Pin_1.5x0.8mm -> myLib:Pad_3Pin_1.5x0.8mm
- C1, C33, C34, C37, C38: value 4.7uF -> 100nF
- C10, C54, C69: value 0.1uF -> 100nF
- C11: value 12pF -> 100nF
- C12, C13: value 12pF -> 1uF
- C14: value 12pF -> 4.7uF
- C15: value 1.0uF -> 1uF
- C16, C21: value 1.0uF -> 4.7uF
- C17, C20, C55, C56, C58: value 100nF -> 1uF
- C19: value 100nF -> 2.2nF
- C2: value 4.7uF -> 0.1uF
- C22: value 1.0uF -> 0.1uF
- C23: value 2.2nF -> 0.1uF
- C24: value 2.2nF -> 10uF
- C25, C26, C27, C28: value 100nF -> 10uF
- C29, C32: value 1.0uF -> 47uF
- C3, C4, C5: value 10uF -> N.M.
- C30, C31: value 1.0uF -> 100nF
- C35, C36: value N.C. -> 100nF
- C39: value N.C. -> 0.1uF
- C40: value 0.7pF -> 100nF
- C41: value N.C. -> N.M.
- C42: value 0.7pF -> 30pF
- C43, C44: value 100nF -> N.M.
- C45: value 1.0uF -> 30pF
- C46: value 1.0uF -> 0.7pF
- C47, C48: value 100nF -> 12pF
- C49, C50, C51: value 100nF -> 30pF
- C57: value 100nF -> 4.7uF
- C59: value 0.1uF -> 4.7uF
- C6: value 10uF -> 0.7pF
- C60, C63: value 0.1uF -> 1uF
- C61, C68: value 30pF -> 100nF
- C62: value 30pF -> 2.2nF
- C64: value 10uF -> 4.7uF
- C65: value 47uF -> 10uF
- C66, C67: value 30pF -> 10uF
- C7, C8: value 10uF -> 12pF
- C70: value 10uF -> 100nF
- C71: value 47uF -> 100nF
- J10: value Low-V -> Prog
- J2: value USB_C_Receptacle_USB2.0_16P -> Touch Pads; footprint Connector_USB:USB_C_Receptacle_GCT_USB4110 -> myLib:Pad_3Pin_1.5x0.8mm
- J3: value Touch Pads -> UART; footprint myLib:Pad_1Pin_2x1.2mm -> myLib:Pad_3Pin_1.5x0.8mm
- J4: value Touch Pads -> Prog; footprint myLib:Pad_1Pin_2x1.2mm -> myLib:Pad_prog_4Pad
- J5: value UART -> Touch Pads
- J6: value UART -> High-V; footprint myLib:Pad_3Pin_1.5x0.8mm -> myLib:Pad_prog_4Pad
- J7: value Prog -> USB_C_Receptacle_USB2.0_16P; footprint myLib:Pad_prog_4Pad -> Connector_USB:USB_C_Receptacle_GCT_USB4110
- J8: value Prog -> Low-V
- J9: value High-V -> Low-V-TH; footprint myLib:Pad_prog_4Pad -> Connector_PinHeader_2.54mm:PinHeader_1x05_P2.54mm_Vertical
- L1: value 2.2uH -> N.M.
- L2: value 2.2uH -> 2.2nH
- L5: value 10uH -> 2.2uH
- L6: value 10uH -> N.M.
- L8: value 2.2nH -> 10uH
- LS2: value SPH18R1LM4H-1-8 -> Boneconduction; footprint myLib:MIC_SPH18R1LM4H_KNO -> myLib:Pad_2Pin_1.5x0.8mm
- LS6: value Boneconduction -> SPH18R1LM4H-1-8; footprint myLib:Pad_2Pin_1.5x0.8mm -> myLib:MIC_SPH18R1LM4H_KNO
- R1: value 1K5R -> 75k
- R10, R9: value 5K1R -> 4k7
- R11, R12: value 5K1R -> 1K5R
- R13: value 4.7k -> 75k
- R14, R15: value 4.7k -> 1K5
- R16: value 4.7k -> 1K8
- R17: value 2R2 -> 1K8
- R18: value 2R2 -> 1K5
- R19: value 75k -> 1K8
- R2, R3: value 1K5R -> 5K1R
- R20: value 75k -> 5K1R
- R21: value 1K5 -> 5K1R
- R23: value 1K8 -> 1K5
- R25: value 1K5 -> 1K8
- R26: value 1K8 -> 2R2
- R27: value N.C. -> 5K1R
- R28: value 1K5 -> 10K
- R29: value 1K5 -> 4k7
- R30: value 1K8 -> 4k7
- R31: value 1K8 -> 1K5R
- R32: value N.C. -> 1K5R
- R4: value 1K5R -> 2R2
- R6: value 5K1R -> 10K
- R7, R8: value 10K -> N.C.
- U1: value NPM1100-CAAA-R7 -> BMA400; footprint myLib:NPM1100-CAAA-BGA25C40P5X5_207X207X52N -> myLib:QFN_BMA400_BOS
- U10: value MAX98357AEWL_T -> NPM1100-CAAA-R7; footprint myLib:MAX98357A_BGA9N40P3X3_134X143X69N -> myLib:NPM1100-CAAA-BGA25C40P5X5_207X207X52N
- U2: value NPM1100-CAAA-R7 -> MPR121QR2; footprint myLib:NPM1100-CAAA-BGA25C40P5X5_207X207X52N -> myLib:MPR121
- U3: value NRF5340-CLAA-R -> NRF5340-QKAA-R
- U4: value NRF5340-CLAA-R -> NPM1100-CAAA-R7; footprint myLib:NRF5340 -> myLib:NPM1100-CAAA-BGA25C40P5X5_207X207X52N
- U5, U6: value BMA400 -> MAX98357AEWL_T; footprint myLib:QFN_BMA400_BOS -> myLib:MAX98357A_BGA9N40P3X3_134X143X69N
- U8: value MPR121QR2 -> BMA400; footprint myLib:MPR121 -> myLib:QFN_BMA400_BOS
- U9: value MAX98357AEWL_T -> NRF5340-QKAA-R; footprint myLib:MAX98357A_BGA9N40P3X3_134X143X69N -> myLib:NRF5340
- Y1: value Crystal -> 32MHz; footprint myLib:Crystal_24MHz-ECS-240-12-37B-CKY-TR -> myLib:ECS-160-10-37-JTN-TR_ECS
- Y2: value Crystal -> 32.768kHz
- moved U1 680.6 mm to (-147.1, 54.4)
- moved J3 679.2 mm to (-140.1, 35.6)
- moved U5 678.1 mm to (-142.1, 51.3)
- moved C71 671.3 mm to (-111.0, 90.6)
- moved BT1 667.4 mm to (-147.7, 35.6)
- moved D1 666.0 mm to (-98.3, 95.7)
- moved D3 666.0 mm to (-98.3, 100.9)
- moved J5 665.4 mm to (-137.6, 35.6)
- moved Y1 664.6 mm to (-125.1, 55.3)
- moved U7 663.9 mm to (-135.7, 52.5)
- moved LS1 663.0 mm to (-125.3, 46.8)
- moved U3 663.0 mm to (-141.4, 40.6)
- moved U9 661.4 mm to (-141.4, 46.2)
- moved LS6 660.6 mm to (-125.3, 51.3)
- moved C57 659.7 mm to (-111.0, 65.5)
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Connections:
- C1 pad 1: GND -> VDD
- C1 pad 2: +3.3V -> GND
- C10 pad 1: VDD -> GND
- C10 pad 2: GND -> VDD
- C11 pad 1: Net-(U3-XC2) -> VDD
- C12 pad 1: Net-(U3-XC1) -> VDD
- C13 pad 1: Net-(U4-XC2) -> Net-(U3A-DECR)
- C14 pad 1: Net-(U4-XC1) -> Net-(U3A-VBUS)
- C15 pad 1: Net-(U3-DECD) -> VDD
- C16 pad 1: Net-(U4-DECD) -> Net-(U3A-DECUSB)
- C17 pad 1: GND -> Net-(U3A-DECD)
- C17 pad 2: Net-(C17-Pad2) -> GND
- C18 pad 1: GND -> Net-(U3A-DECN)
- C18 pad 2: Net-(C18-Pad2) -> GND
- C19 pad 1: GND -> Net-(U3A-DECR)
- C19 pad 2: Net-(C19-Pad2) -> GND
- C2 pad 1: GND -> Net-(U2-VREG)
- C2 pad 2: +3.3V -> GND
- C20 pad 1: GND -> Net-(U3A-DECA)
- C20 pad 2: Net-(C20-Pad2) -> GND
- C21 pad 2: Net-(U3-DECR) -> +3.3V
- C22 pad 1: GND -> +3.3V
- C22 pad 2: Net-(U4-DECR) -> GND
- C23 pad 1: GND -> +3.3V
- C23 pad 2: Net-(U3-DECR) -> GND
- C24 pad 1: GND -> +3.3V
- C24 pad 2: Net-(U4-DECR) -> GND
- C25 pad 1: GND -> +3.3V
- C25 pad 2: Net-(C25-Pad2) -> GND
- C26 pad 2: Net-(C26-Pad2) -> VBUS
- C27 pad 2: Net-(U3-DECN) -> VDD
- C28 pad 2: Net-(U4-DECN) -> Net-(U4-DEC)
- C29 pad 1: GND -> +3.3V
- C29 pad 2: Net-(U3-DECA) -> GND
- C3 pad 1: GND -> Net-(C3-Pad1)
- C3 pad 2: VBUS -> GND
- C30 pad 1: GND -> VDD
- C30 pad 2: Net-(U4-DECA) -> GND
- C32 pad 1: VDD -> +3.3V
- C33 pad 1: Net-(U3-DECUSB) -> VDD
- C34 pad 1: Net-(U4-DECUSB) -> VDD
- C35 pad 1: Net-(C35-Pad1) -> VDD
- C35 pad 2: Net-(U3-ANT) -> GND
- C36 pad 1: Net-(C36-Pad1) -> VDD
- C36 pad 2: Net-(U4-ANT) -> GND
- C37 pad 1: Net-(U3-VBUS) -> VDD
- C38 pad 1: Net-(U4-VBUS) -> VDD
- C39 pad 1: /RF -> Net-(U7-VREG)
- C4 pad 1: GND -> Net-(C3-Pad1)
- C4 pad 2: VBUS -> GND
- C40 pad 1: Net-(C35-Pad1) -> VDD
- C41 pad 1: /RF -> Net-(C41-Pad1)
- C42 pad 1: Net-(C36-Pad1) -> /A1
- C42 pad 2: GND -> /B1
- C43 pad 1: GND -> Net-(C41-Pad1)
- C43 pad 2: Net-(C43-Pad2) -> GND
- C44 pad 1: GND -> Net-(AE2-A)
- C44 pad 2: Net-(C44-Pad2) -> GND
- C45 pad 1: VDD -> /A4
- C45 pad 2: GND -> /B4
- C46 pad 1: VDD -> Net-(U9D-ANT)
- C47 pad 1: GND -> Net-(U9D-XC2)
- C47 pad 2: Net-(C47-Pad2) -> GND
- C48 pad 1: GND -> Net-(U9D-XC1)
- C48 pad 2: Net-(C48-Pad2) -> GND
- C49 pad 1: VDD -> /A3
- C49 pad 2: GND -> /B3
- C5 pad 1: GND -> Net-(AE1-A)
- C5 pad 2: VDD -> GND
- C50 pad 1: VDD -> /A2
- C50 pad 2: GND -> /B2
- C51 pad 1: GND -> /A5
- C51 pad 2: VDD -> /B5
- C53 pad 1: GND -> VDD
- C53 pad 2: /nRESET -> GND
- C54 pad 1: GND -> VDD
- C54 pad 2: /nRESET -> GND
- C55 pad 1: GND -> VDD
- C55 pad 2: Net-(C55-Pad2) -> GND
- C56 pad 1: GND -> Net-(U9A-DECR)
- C56 pad 2: Net-(C56-Pad2) -> GND
- C57 pad 1: VDD -> Net-(U9A-VBUS)
- C59 pad 1: Net-(U7-VREG) -> Net-(U9A-DECUSB)
- C6 pad 1: GND -> Net-(U3D-ANT)
- C6 pad 2: VDD -> GND
- C60 pad 1: Net-(U8-VREG) -> Net-(U9A-DECD)
- C61 pad 1: /A1 -> Net-(U9A-DECN)
- C61 pad 2: /B1 -> GND
- C62 pad 1: /A2 -> Net-(U9A-DECR)
- C62 pad 2: /B2 -> GND
- C63 pad 1: +3.3V -> Net-(U9A-DECA)
- C64 pad 1: +3.3V -> GND
- C64 pad 2: GND -> +3.3V
- C65 pad 1: +3.3V -> GND
- C65 pad 2: GND -> VBUS
- C66 pad 1: /A3 -> GND
- C66 pad 2: /B3 -> VDD
- C67 pad 1: /A4 -> GND
- C67 pad 2: /B4 -> Net-(U10-DEC)
- C68 pad 1: /A5 -> VDD
- C68 pad 2: /B5 -> GND
- C69 pad 1: +3.3V -> VDD
- C7 pad 1: GND -> Net-(U3D-XC2)
- C7 pad 2: Net-(U1-DEC) -> GND
- C70 pad 1: +3.3V -> VDD
- C71 pad 1: +3.3V -> VDD
- C8 pad 1: GND -> Net-(U3D-XC1)
- C8 pad 2: Net-(U2-DEC) -> GND
- J10 pad 1: /B1 -> VDD
- J10 pad 2: /B2 -> /SWDIO
- J10 pad 3: /B3 -> /SWDCLK
- J10 pad 4: /B4 -> GND
- J10 pad 5: /B5 -> /nRESET
- J3 pad 1: Net-(J3-Pin_1) -> /TX
- J4 pad 1: Net-(J4-Pin_1) -> VDD
- J5 pad 1: /TX -> Net-(J5-Pin_1)
- J5 pad 2: /RX -> Net-(J5-Pin_2)
- J5 pad 3: GND -> Net-(J5-Pin_3)
- J6 pad 1: /TX -> /A1
- J6 pad 2: /RX -> /A2
- J6 pad 3: GND -> /A3
- J8 pad 1: VDD -> /B1
- J8 pad 2: /SWDIO -> /B2
- J8 pad 3: /SWDCLK -> /B3
- J8 pad 4: GND -> /B4
- J8 pad 5: /nRESET -> /B5
- J9 pad 1: /A1 -> /B5
- J9 pad 2: /A2 -> /B4
- J9 pad 3: /A3 -> /B3
- J9 pad 4: /A4 -> /B2
- J9 pad 5: /A5 -> /B1
- L1 pad 1: VDD -> Net-(AE1-A)
- L1 pad 2: Net-(U1-SW) -> Net-(C3-Pad1)
- L2 pad 1: VDD -> Net-(C3-Pad1)
- L2 pad 2: Net-(U2-SW) -> Net-(U3D-ANT)
- L3 pad 1: Net-(U3-DCCD) -> Net-(U3A-DECR)
- L3 pad 2: Net-(U3-DECD) -> Net-(U3A-DCCR)
- L4 pad 1: Net-(U4-DCCD) -> Net-(U3A-DECD)
- L4 pad 2: Net-(U4-DECD) -> Net-(U3A-DCCD)
- L5 pad 1: Net-(U3-DCC) -> VDD
- L5 pad 2: Net-(U3-DECR) -> Net-(U4-SW)
- L6 pad 1: Net-(U4-DCC) -> Net-(AE2-A)
- L6 pad 2: Net-(U4-DECR) -> Net-(C41-Pad1)
- L7 pad 1: /RF -> Net-(C41-Pad1)
- L7 pad 2: Net-(C35-Pad1) -> Net-(U9D-ANT)
- L8 pad 1: /RF -> Net-(U9A-DECR)
- L8 pad 2: Net-(C36-Pad1) -> Net-(U9A-DCCR)
- LS2 pad 1: /MIC_DATA -> Net-(U5-OUTN)
- LS2 pad 2: unconnected-(LS2-SELECT-Pad2) -> Net-(U5-OUTP)
- LS3 pad 1: Net-(U9-OUTN) -> Net-(U5-OUTN)
- LS3 pad 2: Net-(U9-OUTP) -> Net-(U5-OUTP)
- LS4 pad 1: Net-(U9-OUTN) -> Net-(U6-OUTN)
- LS4 pad 2: Net-(U9-OUTP) -> Net-(U6-OUTP)
- LS5 pad 1: Net-(U10-OUTN) -> Net-(U6-OUTN)
- LS5 pad 2: Net-(U10-OUTP) -> Net-(U6-OUTP)
- LS6 pad 1: Net-(U10-OUTN) -> /MIC_DATA
- LS6 pad 2: Net-(U10-OUTP) -> unconnected-(LS6-SELECT-Pad2)
- R1 pad 1: Net-(D1-A) -> Net-(U2-REXT)
- R1 pad 2: VSYS -> GND
- R10 pad 1: GND -> /I2C_SDA
- R10 pad 2: Net-(J2-CC1) -> VDD
- R11 pad 1: GND -> Net-(D2-A)
- R11 pad 2: Net-(J1-CC2) -> VSYS
- R12 pad 1: GND -> Net-(D1-A)
- R12 pad 2: Net-(J2-CC2) -> VSYS
- R13 pad 1: VDD -> Net-(U7-REXT)
- R13 pad 2: /I2C_SCL -> GND
- R14 pad 1: VDD -> /A1
- R14 pad 2: /I2C_SCL -> Net-(R14-Pad2)
- R15 pad 1: VDD -> /A4
- R15 pad 2: /I2C_SDA -> Net-(R15-Pad2)
- R16 pad 1: VDD -> /B1
- R16 pad 2: /I2C_SDA -> Net-(R14-Pad2)
- R17 pad 1: Net-(U3-VBUS) -> /B4
- R17 pad 2: VBUS -> Net-(R15-Pad2)
- R18 pad 1: Net-(U4-VBUS) -> /A3
- R18 pad 2: VBUS -> Net-(R18-Pad2)
- R19 pad 1: Net-(U7-REXT) -> /B3
- R19 pad 2: GND -> Net-(R18-Pad2)
- R2 pad 1: Net-(D2-A) -> GND
- R2 pad 2: VSYS -> Net-(J1-CC1)
- R20 pad 1: Net-(U8-REXT) -> GND
- R20 pad 2: GND -> Net-(J7-CC1)
- R21 pad 1: /A1 -> GND
- R21 pad 2: Net-(R21-Pad2) -> Net-(J7-CC2)
- R23 pad 1: /B1 -> /A5
- R23 pad 2: Net-(R21-Pad2) -> Net-(R23-Pad2)
- R25 pad 1: /A3 -> /B5
- R25 pad 2: Net-(R25-Pad2) -> Net-(R23-Pad2)
- R26 pad 1: /B3 -> Net-(U9A-VBUS)
- R26 pad 2: Net-(R25-Pad2) -> VBUS
- R27 pad 2: Net-(U9-GAIN_SLOT) -> Net-(U10-ICHG)
- R28 pad 1: /A4 -> GND
- R28 pad 2: Net-(R28-Pad2) -> Net-(U10-NTC)
- R29 pad 1: /A5 -> /I2C_SCL
- R29 pad 2: Net-(R29-Pad2) -> VDD
- R3 pad 1: Net-(D3-A) -> GND
- R3 pad 2: VSYS -> Net-(J1-CC2)
- R30 pad 1: /B4 -> /I2C_SDA
- R30 pad 2: Net-(R28-Pad2) -> VDD
- R31 pad 1: /B5 -> Net-(D4-A)
- R31 pad 2: Net-(R29-Pad2) -> VSYS
- R32 pad 1: GND -> Net-(D3-A)
- R32 pad 2: Net-(U10-GAIN_SLOT) -> VSYS
- R4 pad 1: Net-(D4-A) -> Net-(U3A-VBUS)
- R4 pad 2: VSYS -> VBUS
- R5 pad 2: Net-(U1-ICHG) -> Net-(U4-ICHG)
- R6 pad 2: Net-(U2-ICHG) -> Net-(U4-NTC)
- R7 pad 2: Net-(U1-NTC) -> Net-(U5-GAIN_SLOT)
- R8 pad 2: Net-(U2-NTC) -> Net-(U6-GAIN_SLOT)
- R9 pad 1: GND -> /I2C_SCL
- R9 pad 2: Net-(J1-CC1) -> VDD
- U10 pad A1: /SD_MODE -> /D-
- U10 pad A2: +3.3V -> /D+
- U10 pad A3: Net-(U10-OUTP) -> Net-(U10-DEC)
- U10 pad B1: /SDOUT -> VBUS
- U10 pad B2: Net-(U10-GAIN_SLOT) -> VBUS
- U10 pad B3: Net-(U10-OUTN) -> GND
- U10 pad C1: /SCK -> VSYS
- U10 pad C2: GND -> VSYS
- U10 pad C3: /LRCLK -> VDD
- U3 pad A1: Net-(U3-XC1) -> unconnected-(U3D-NC-PadA1)
- U3 pad A11: /D- -> (no net)
- U3 pad A12: /D+ -> (no net)
- U3 pad A2: Net-(U3-XC2) -> (no net)
- U3 pad A3: Net-(C19-Pad2) -> (no net)
- U3 pad A5: GND -> Net-(U3A-VBUS)
- U3 pad A7: Net-(U3-DECD) -> (no net)
- U3 pad A9: Net-(U3-DCCD) -> (no net)
- U3 pad B1: Net-(U3-DECR) -> (no net)
- U3 pad B10: VDD -> Net-(U3A-DCCD)
- U3 pad B11: Net-(U3-VBUS) -> (no net)
- U3 pad B12: VDD -> GND
- U3 pad B2: GND -> /D+
- U3 pad B4: Net-(U3-DECR) -> /D-
- U3 pad B5: Net-(U3-DECN) -> (no net)
- U3 pad B6: Net-(U3-DCC) -> Net-(U3A-DECUSB)
- U3 pad B7: VDD -> (no net)
- U3 pad B8: Net-(U3-DECA) -> VDD
- U3 pad B9: GND -> (no net)
- U3 pad C10: unconnected-(U3-P1.15-PadC10) -> (no net)
- U3 pad C11: Net-(U3-DECUSB) -> (no net)
- U3 pad C2: GND -> (no net)
- U3 pad C4: unconnected-(U3-P0.30-PadC4) -> (no net)
- U3 pad C5: unconnected-(U3-P0.31-PadC5) -> (no net)
- U3 pad C6: unconnected-(U3-P1.11-PadC6) -> (no net)
- U3 pad C7: /SCK -> (no net)
- U3 pad C8: /LRCLK -> (no net)
- U3 pad C9: /SDOUT -> (no net)
- U3 pad D1: Net-(U3-ANT) -> (no net)
- U3 pad D10: unconnected-(U3-P1.00-PadD10) -> (no net)
- U3 pad D11: unconnected-(U3-DCCH-PadD11) -> (no net)
- U3 pad D12: GND -> (no net)
- U3 pad D2: Net-(C43-Pad2) -> unconnected-(U3D-NC-PadD2)
- U3 pad E10: unconnected-(U3-P1.01-PadE10) -> (no net)
- U3 pad E11: VDD -> (no net)
- U3 pad E2: unconnected-(U3-P0.29-PadE2) -> (no net)
- U3 pad E3: unconnected-(U3-P0.28/AIN7-PadE3) -> (no net)
- U3 pad E4: unconnected-(U3-P1.10-PadE4) -> (no net)
- U3 pad E5: GND -> (no net)
- U3 pad E6: GND -> (no net)
- U3 pad E7: GND -> (no net)
- U3 pad E8: GND -> (no net)
- U3 pad F1: /SWDIO -> (no net)
- U3 pad F10: /I2C_SDA -> (no net)
- U3 pad F11: unconnected-(U3-P0.00/XL1-PadF11) -> (no net)
- U3 pad F12: unconnected-(U3-P0.01/XL2-PadF12) -> (no net)
- U3 pad F2: /SWDCLK -> unconnected-(U3D-NC-PadF2)
- U3 pad F3: unconnected-(U3-P1.08-PadF3) -> (no net)
- U3 pad F5: GND -> (no net)
- U3 pad F6: GND -> (no net)
- U3 pad F7: GND -> (no net)
- U3 pad F8: GND -> (no net)
- U3 pad G10: /I2C_SCL -> (no net)
- U3 pad G11: unconnected-(U3-P0.02/NFC1-PadG11) -> (no net)
- U3 pad G2: /nRESET -> (no net)
- U3 pad G3: unconnected-(U3-P1.07-PadG3) -> (no net)
- U3 pad G5: GND -> (no net)
- U3 pad G6: GND -> (no net)
- U3 pad G7: GND -> (no net)
- U3 pad G8: GND -> (no net)
- U3 pad H1: unconnected-(U3-P0.27/AIN6-PadH1) -> (no net)
- U3 pad H10: /INT1 -> (no net)
- U3 pad H11: Net-(C25-Pad2) -> (no net)
- U3 pad H12: unconnected-(U3-P0.03/NFC2-PadH12) -> (no net)
- U3 pad H2: unconnected-(U3-P1.09-PadH2) -> GND
- U3 pad H3: unconnected-(U3-P0.23-PadH3) -> (no net)
- U3 pad J10: /INT2 -> (no net)
- U3 pad J11: unconnected-(U3-P1.02/TWI-PadJ11) -> (no net)
- U3 pad J2: /MIC_CLOCK -> (no net)
- U3 pad J3: unconnected-(U3-P1.06-PadJ3) -> (no net)
- U3 pad J4: unconnected-(U3-P0.21-PadJ4) -> (no net)
- U3 pad J5: unconnected-(U3-P0.19-PadJ5) -> (no net)
- U3 pad J6: unconnected-(U3-P0.12/TRACECLK/DCX-PadJ6) -> (no net)
- U3 pad J7: unconnected-(U3-P0.11/TRACEDATA0/CSN-PadJ7) -> (no net)
- U3 pad J8: unconnected-(U3-P0.10/TRACEDATA1/MISO-PadJ8) -> (no net)
- U3 pad J9: unconnected-(U3-P0.09/TRACEDATA2/MOSI-PadJ9) -> (no net)
- U3 pad K1: Net-(C55-Pad2) -> (no net)
- U3 pad K10: unconnected-(U3-P0.13/IO0-PadK10) -> (no net)
- U3 pad K11: unconnected-(U3-AVSS-PadK11) -> (no net)
- U3 pad K12: unconnected-(U3-P1.03/TWI-PadK12) -> (no net)
- U3 pad K3: unconnected-(U3-P1.04-PadK3) -> (no net)
- U3 pad K4: /ISET -> (no net)
- U3 pad K5: /SD_MODE -> (no net)
- U3 pad K6: GND -> (no net)
- U3 pad K7: unconnected-(U3-P0.18/CSN-PadK7) -> (no net)
- U3 pad K8: unconnected-(U3-P0.16/IO3-PadK8) -> (no net)
- U3 pad K9: unconnected-(U3-P0.14/IO1-PadK9) -> (no net)
- U3 pad L1: /MIC_DATA -> VDD
- U3 pad L11: Net-(C17-Pad2) -> (no net)
- U3 pad L12: unconnected-(U3-P0.08/TRACEDATA3/SCK-PadL12) -> (no net)
- U3 pad L3: unconnected-(U3-P1.05-PadL3) -> (no net)
- U3 pad L5: Net-(C47-Pad2) -> (no net)
- U3 pad L7: unconnected-(U3-P0.17/SCK-PadL7) -> (no net)
- U3 pad L9: unconnected-(U3-P0.15/IO2-PadL9) -> (no net)
- U4 pad A1: Net-(U4-XC1) -> /D-
- U4 pad A2: Net-(U4-XC2) -> /D+
- U4 pad A3: Net-(C20-Pad2) -> Net-(U4-DEC)
- U4 pad B1: Net-(U4-DECR) -> VBUS
- U4 pad B2: GND -> VBUS
- U4 pad B4: Net-(U4-DECR) -> GND
- U4 pad B5: Net-(U4-DECN) -> VDD
- U4 pad C2: GND -> VSYS
- U4 pad C4: unconnected-(U4-P0.30-PadC4) -> GND
- U4 pad C5: unconnected-(U4-P0.31-PadC5) -> GND
- U4 pad D1: Net-(U4-ANT) -> +3.3V
- U4 pad D2: Net-(C44-Pad2) -> +3.3V
- U4 pad E2: unconnected-(U4-P0.29-PadE2) -> Net-(U4-ICHG)
- U4 pad E3: unconnected-(U4-P0.28/AIN7-PadE3) -> Net-(D1-K)
- U4 pad E4: unconnected-(U4-P1.10-PadE4) -> Net-(D2-K)
- U7 pad 10: Net-(J3-Pin_3) -> Net-(J5-Pin_3)
- U7 pad 8: Net-(J3-Pin_1) -> Net-(J5-Pin_1)
- U7 pad 9: Net-(J3-Pin_2) -> Net-(J5-Pin_2)
- U8 pad 1: /IRQ -> GND
- U8 pad 10: Net-(J4-Pin_3) -> VDD
- U8 pad 12: unconnected-(U8-ELE4-Pad12) -> /I2C_SCL
- U8 pad 2: /I2C_SCL -> /I2C_SDA
- U8 pad 3: /I2C_SDA -> VDD
- U8 pad 4: GND -> unconnected-(U8-NC-Pad4)
- U8 pad 5: Net-(U8-VREG) -> /INT1
- U8 pad 6: GND -> /INT2
- U8 pad 7: Net-(U8-REXT) -> VDD
- U8 pad 8: Net-(J4-Pin_1) -> GND
- U8 pad 9: Net-(J4-Pin_2) -> GND
- U9 pad A1: /SD_MODE -> unconnected-(U9D-NC-PadA1)
- U9 pad A2: +3.3V -> (no net)
- U9 pad A3: Net-(U9-OUTP) -> (no net)
- U9 pad B1: /SDOUT -> (no net)
- U9 pad B2: Net-(U9-GAIN_SLOT) -> /D+
- U9 pad C2: GND -> (no net)
- Y1 pad 1: Net-(U3-XC2) -> Net-(U3D-XC1)
- Y1 pad 2: Net-(U3-XC1) -> Net-(U3D-XC2)
- Y2 pad 1: Net-(U4-XC2) -> Net-(U3B-P0.01/XL2)
- Y2 pad 2: GND -> Net-(U3B-P0.00/XL1)
- Y2 pad 3: Net-(U4-XC1) -> (no net)
- Y2 pad 4: GND -> (no net)
Other:
- board text removed: "A3"
- board text removed: "B1"
- board text removed: "B10"
- board text removed: "B5"
- board text removed: "B7"
- board text removed: "B8"
- board text removed: "D2"
- board text removed: "H11"
- board text removed: "K1"
- board text removed: "L11"
- board text removed: "L5"

Commit message: update 2
Parts:
- U3, U9: footprint myLib:NRF5340 -> Package_DFN_QFN:Nordic_AQFN-94-1EP_7x7mm_P0.4mm
- moved U8 24.4 mm to (-165.8, 42.3)
- moved U3 15.0 mm to (-155.7, 36.1)
- moved U9 13.9 mm to (-154.8, 49.9)
Connections:
- U1 pad 5: /INT1 -> INT1
- U8 pad 5: /INT1 -> INT1
