File: hardware/kicad/ver_1.0/MSBE_V3.kicad_pcb (KiCad board)
At the start: 4 copper layers, 156 parts, among them J1 USB_C_Receptacle_USB2.0_16P, J10 Prog, J11 UART, J2 Touch Pads, J3 UART, J4 Prog, J5 Touch Pads, J6 High-V, J7 USB_C_Receptacle_USB2.0_16P, J8 Low-V, J9 Low-V-TH, U1 BMA400, U10 NPM1100-CAAA-R7, U2 MPR121QR2, U3 NRF5340-QKAA-R, U4 NPM1100-CAAA-R7, U5 MAX98357AEWL_T, U6 MAX98357AEWL_T, U7 MPR121QR2, U8 BMA400, U9 NRF5340-QKAA-R, Y1 32MHz, Y2 32.768kHz, Y3 32MHz, Y4 32.768kHz

Commit message: izmene 7.11
Parts:
- added R33: 680k, Resistor_SMD:R_0603_1608Metric, F.Cu at (201.8, 146.1)
- added R34: 680k, Resistor_SMD:R_0603_1608Metric, F.Cu at (506.7, 43.1)
- moved C23 634.7 mm to (532.7, 3.57)
- moved C25 634.7 mm to (532.7, 6.08)
- moved C32 634.7 mm to (532.7, 8.59)
- moved R8 634.7 mm to (548.7, 23.7)
- moved LS4 621.9 mm to (493.0, -4.91)
- moved LS5 621.9 mm to (495.6, -4.91)
- moved U6 621.9 mm to (478.4, 15.8)
- moved AE2 567.5 mm to (452.3, -10.6)
- moved C39 567.5 mm to (453.5, -35.6)
- moved C40 567.5 mm to (453.5, -48.1)
- moved C41 567.5 mm to (449.5, -40.6)
- moved C42 567.5 mm to (453.5, -33.0)
- moved C43 567.5 mm to (449.5, -38.1)
- moved C44 567.5 mm to (449.5, -35.6)
- moved C45 567.5 mm to (453.5, -18.0)
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Connections:
- U1 pad 5: INT1 -> /INT1
- U3 pad A17: /LRCLK -> (no net)
- U3 pad A25: GND -> (no net)
- U3 pad AA1: GND -> (no net)
- U3 pad AA31: /SWDIO -> (no net)
- U3 pad AB2: INT1 -> (no net)
- U3 pad AC31: /nRESET -> (no net)
- U3 pad AD2: /INT2 -> (no net)
- U3 pad AE1: unconnected-(U3C-P1.02/TWI-PadAE1) -> (no net)
- U3 pad AE31: unconnected-(U3B-P0.28/AIN7-PadAE31) -> (no net)
- U3 pad AF2: unconnected-(U3C-P1.03/TWI-PadAF2) -> (no net)
- U3 pad AG31: unconnected-(U3A-DECF-PadAG31) -> (no net)
- U3 pad AH2: unconnected-(U3B-P0.08/TRACEDATA3/SCK-PadAH2) -> (no net)
- U3 pad AJ1: unconnected-(U3B-P0.09/TRACEDATA2/MOSI-PadAJ1) -> (no net)
- U3 pad AK10: unconnected-(U3B-P0.15/IO2-PadAK10) -> (no net)
- U3 pad AK12: unconnected-(U3B-P0.17/SCK-PadAK12) -> (no net)
- U3 pad AK14: unconnected-(U3B-P0.18/CSN-PadAK14) -> (no net)
- U3 pad AK16: /SD_MODE -> (no net)
- U3 pad AK18: /ISET -> (no net)
- U3 pad AK2: unconnected-(U3B-P0.10/TRACEDATA1/MISO-PadAK2) -> (no net)
- U3 pad AK20: unconnected-(U3B-P0.23-PadAK20) -> (no net)
- U3 pad AK22: unconnected-(U3C-P1.05-PadAK22) -> (no net)
- U3 pad AK24: unconnected-(U3C-P1.07-PadAK24) -> (no net)
- U3 pad AK26: unconnected-(U3C-P1.09-PadAK26) -> (no net)
- U3 pad AK28: /MIC_DATA -> (no net)
- U3 pad AK30: unconnected-(U3B-P0.27/AIN6-PadAK30) -> (no net)
- U3 pad AK4: unconnected-(U3B-P0.11/TRACEDATA0/CSN-PadAK4) -> (no net)
- U3 pad AK6: unconnected-(U3B-P0.12/TRACECLK/DCX-PadAK6) -> (no net)
- U3 pad AK8: unconnected-(U3B-P0.14/IO1-PadAK8) -> (no net)
- U3 pad AL13: unconnected-(U3B-P0.19-PadAL13) -> (no net)
- U3 pad AL15: unconnected-(U3B-P0.21-PadAL15) -> (no net)
- U3 pad AL19: unconnected-(U3C-P1.04-PadAL19) -> (no net)
- U3 pad AL21: unconnected-(U3C-P1.06-PadAL21) -> (no net)
- U3 pad AL23: unconnected-(U3C-P1.08-PadAL23) -> (no net)
- U3 pad AL27: unconnected-(U3B-P0.24-PadAL27) -> (no net)
- U3 pad AL29: /MIC_CLOCK -> (no net)
- U3 pad AL5: unconnected-(U3B-P0.13/IO0-PadAL5) -> (no net)
- U3 pad AL9: unconnected-(U3B-P0.16/IO3-PadAL9) -> (no net)
- U3 pad B14: unconnected-(U3C-P1.15-PadB14) -> (no net)
- U3 pad B16: /SDOUT -> (no net)
- U3 pad B18: /SCK -> (no net)
- U3 pad B20: unconnected-(U3C-P1.11-PadB20) -> (no net)
- U3 pad B22: unconnected-(U3B-P0.31-PadB22) -> (no net)
- U3 pad B24: unconnected-(U3B-P0.30-PadB24) -> (no net)
- U3 pad B26: GND -> (no net)
- U3 pad B30: Net-(U3D-XC2) -> (no net)
- U3 pad C31: Net-(U3D-XC1) -> (no net)
- U3 pad G1: GND -> (no net)
- U3 pad J1: unconnected-(U3A-DCCH-PadJ1) -> (no net)
- U3 pad J31: GND -> (no net)
- U3 pad L31: Net-(U3D-ANT) -> (no net)
- U3 pad M2: unconnected-(U3C-P1.00-PadM2) -> (no net)
- U3 pad P2: unconnected-(U3C-P1.01-PadP2) -> (no net)
- U3 pad R31: unconnected-(U3C-P1.10-PadR31) -> (no net)
- U3 pad T2: unconnected-(U3D-NC-PadT2) -> (no net)
- U3 pad U31: unconnected-(U3B-P0.29-PadU31) -> (no net)
- U3 pad V2: /I2C_SCL -> (no net)
- U3 pad W1: GND -> (no net)
- U3 pad W31: /SWDCLK -> (no net)
- U3 pad Y2: /I2C_SDA -> (no net)
- U8 pad 5: INT1 -> /INT1
- U9 pad A13: Net-(U9A-DECA) -> (no net)
- U9 pad A15: Net-(U9A-DECD) -> (no net)
- U9 pad A17: /LRCLK -> (no net)
- U9 pad A19: VDD -> (no net)
- U9 pad A21: Net-(U9A-DCCR) -> (no net)
- U9 pad A23: Net-(U9A-DECN) -> (no net)
- U9 pad A25: GND -> (no net)
- U9 pad A27: Net-(U9A-DECR) -> (no net)
- U9 pad AA1: GND -> (no net)
- U9 pad AA31: /SWDIO -> (no net)
- U9 pad AB2: INT1 -> (no net)
- U9 pad AC1: VDD -> (no net)
- U9 pad AC31: /nRESET -> (no net)
- U9 pad AD2: /INT2 -> (no net)
- U9 pad AE1: unconnected-(U9C-P1.02/TWI-PadAE1) -> (no net)
- U9 pad AE31: unconnected-(U9B-P0.28/AIN7-PadAE31) -> (no net)
- U9 pad AF2: unconnected-(U9C-P1.03/TWI-PadAF2) -> (no net)
- U9 pad AG1: VDD -> (no net)
- U9 pad AG31: unconnected-(U9A-DECF-PadAG31) -> (no net)
- U9 pad AH2: unconnected-(U9B-P0.08/TRACEDATA3/SCK-PadAH2) -> (no net)
- U9 pad AJ1: unconnected-(U9B-P0.09/TRACEDATA2/MOSI-PadAJ1) -> (no net)
- U9 pad AJ31: VDD -> (no net)
- U9 pad AK10: unconnected-(U9B-P0.15/IO2-PadAK10) -> (no net)
- U9 pad AK12: unconnected-(U9B-P0.17/SCK-PadAK12) -> (no net)
- U9 pad AK14: unconnected-(U9B-P0.18/CSN-PadAK14) -> (no net)
- U9 pad AK16: /SD_MODE -> (no net)
- U9 pad AK18: /ISET -> (no net)
- U9 pad AK2: unconnected-(U9B-P0.10/TRACEDATA1/MISO-PadAK2) -> (no net)
- U9 pad AK20: unconnected-(U9B-P0.23-PadAK20) -> (no net)
- U9 pad AK22: unconnected-(U9C-P1.05-PadAK22) -> (no net)
- U9 pad AK24: unconnected-(U9C-P1.07-PadAK24) -> (no net)
- U9 pad AK26: unconnected-(U9C-P1.09-PadAK26) -> (no net)
- U9 pad AK28: /MIC_DATA -> (no net)
- U9 pad AK30: unconnected-(U9B-P0.27/AIN6-PadAK30) -> (no net)
- U9 pad AK4: unconnected-(U9B-P0.11/TRACEDATA0/CSN-PadAK4) -> (no net)
- U9 pad AK6: unconnected-(U9B-P0.12/TRACECLK/DCX-PadAK6) -> (no net)
- U9 pad AK8: unconnected-(U9B-P0.14/IO1-PadAK8) -> (no net)
- U9 pad AL11: VDD -> (no net)
- U9 pad AL13: unconnected-(U9B-P0.19-PadAL13) -> (no net)
- U9 pad AL15: unconnected-(U9B-P0.21-PadAL15) -> (no net)
- U9 pad AL17: VDD -> (no net)
- U9 pad AL19: unconnected-(U9C-P1.04-PadAL19) -> (no net)
- U9 pad AL21: unconnected-(U9C-P1.06-PadAL21) -> (no net)
- U9 pad AL23: unconnected-(U9C-P1.08-PadAL23) -> (no net)
- U9 pad AL25: VDD -> (no net)
- U9 pad AL27: unconnected-(U9B-P0.24-PadAL27) -> (no net)
- U9 pad AL29: /MIC_CLOCK -> (no net)
- U9 pad AL3: VDD -> (no net)
- U9 pad AL5: unconnected-(U9B-P0.13/IO0-PadAL5) -> (no net)
- U9 pad AL7: VDD -> (no net)
- U9 pad AL9: unconnected-(U9B-P0.16/IO3-PadAL9) -> (no net)
- U9 pad B14: unconnected-(U9C-P1.15-PadB14) -> (no net)
- U9 pad B16: /SDOUT -> (no net)
- U9 pad B18: /SCK -> (no net)
- U9 pad B20: unconnected-(U9C-P1.11-PadB20) -> (no net)
- U9 pad B22: unconnected-(U9B-P0.31-PadB22) -> (no net)
- U9 pad B24: unconnected-(U9B-P0.30-PadB24) -> (no net)
- U9 pad B26: GND -> (no net)
- U9 pad B28: VDD -> (no net)
- U9 pad B30: Net-(U9D-XC2) -> (no net)
- U9 pad C1: VDD -> (no net)
- U9 pad C31: Net-(U9D-XC1) -> (no net)
- U9 pad E1: VDD -> (no net)
- U9 pad E31: VDD -> (no net)
- U9 pad G1: GND -> (no net)
- U9 pad G31: Net-(U9A-DECR) -> (no net)
- U9 pad J1: unconnected-(U9A-DCCH-PadJ1) -> (no net)
- U9 pad J31: GND -> (no net)
- U9 pad L31: Net-(U9D-ANT) -> (no net)
- U9 pad M2: unconnected-(U9C-P1.00-PadM2) -> (no net)
- U9 pad N1: Net-(U9B-P0.00/XL1) -> (no net)
- U9 pad N31: VDD -> (no net)
- U9 pad P2: unconnected-(U9C-P1.01-PadP2) -> (no net)
- U9 pad R1: Net-(U9B-P0.01/XL2) -> (no net)
- U9 pad R31: unconnected-(U9C-P1.10-PadR31) -> (no net)
- U9 pad T2: unconnected-(U9D-NC-PadT2) -> (no net)
- U9 pad U1: VDD -> (no net)
- U9 pad U31: unconnected-(U9B-P0.29-PadU31) -> (no net)
- U9 pad V2: /I2C_SCL -> (no net)
- U9 pad W1: GND -> (no net)
- U9 pad W31: /SWDCLK -> (no net)
- U9 pad Y2: /I2C_SDA -> (no net)

Commit message: done with PCB, need to import to easy eda for better routign
Parts:
- moved J1 197.7 mm to (55.0, 101.2), turned to -90 degrees
- moved R3 178.0 mm to (62.3, 103.6), turned to 180 degrees
- moved R2 177.4 mm to (62.2, 99.3), turned to 180 degrees
- moved R1 173.9 mm to (65.1, 114.6), turned to 180 degrees
- moved R9 167.4 mm to (69.1, 95.6)
- moved R10 167.3 mm to (69.1, 97.4)
- moved C11 165.7 mm to (62.8, 108.8), turned to -90 degrees
- moved C2 165.0 mm to (62.8, 112.3), turned to 90 degrees
- moved R11 163.5 mm to (65.0, 87.5), turned to 90 degrees
- moved R12 162.3 mm to (66.8, 87.5), turned to 90 degrees
- moved R5 159.1 mm to (67.5, 84.1), turned to -90 degrees
- moved R6 157.2 mm to (69.1, 84.1), turned to -90 degrees
- moved D2 154.1 mm to (65.0, 90.6), turned to 90 degrees
- moved D1 152.7 mm to (66.8, 90.6), turned to 90 degrees
- moved L5 151.1 mm to (73.5, 91.5), turned to 90 degrees
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Connections:
- BT1 pad 2: GND -> (no net)
- BT1 pad 3: (no net) -> GND
- U3 pad A17: (no net) -> /LRCLK
- U3 pad AA31: (no net) -> /SWDIO
- U3 pad AB2: (no net) -> /INT1
- U3 pad AC31: (no net) -> /nRESET
- U3 pad AD2: (no net) -> /INT2
- U3 pad B16: (no net) -> /SDOUT
- U3 pad B18: (no net) -> /SCK
- U3 pad B30: (no net) -> Net-(U3D-XC2)
- U3 pad C31: (no net) -> Net-(U3D-XC1)
- U3 pad L31: (no net) -> Net-(U3D-ANT)
- U3 pad M2: (no net) -> /TX
- U3 pad P2: (no net) -> /RX
- U3 pad V2: (no net) -> /I2C_SCL
- U3 pad W31: (no net) -> /SWDCLK
- U3 pad Y2: (no net) -> /I2C_SDA
- Y1 pad 2: Net-(U3D-XC2) -> GND
- Y1 pad 3: (no net) -> Net-(U3D-XC2)
- Y1 pad 4: (no net) -> GND
Other:
- board outline added: 49.3 x 34.5 mm
- copper layers 4 -> 6

Commit message: start of routing
Parts:
- removed AE2: Antenna_Shield, RF_Antenna:Texas_SWRA117D_2.4GHz_Left
- removed BT2: Battery_Cell, myLib:Pad_3Pin_1.5x0.8mm
- removed C22, C39, C53: 0.1uF, Capacitor_SMD:C_0603_1608Metric
- removed C24, C65, C66, C67: 10uF, Capacitor_SMD:C_0603_1608Metric
- removed C29: 47uF, Capacitor_SMD:C_0603_1608Metric
- removed C40, C52, C54, C61, C68, C69, C70, C71, C72, C73, C74, C75: 100nF, Capacitor_SMD:C_0603_1608Metric
- removed C41, C43, C44: N.M., Capacitor_SMD:C_0603_1608Metric
- removed C46: 0.7pF, Capacitor_SMD:C_0603_1608Metric
- removed C47, C48: 12pF, Capacitor_SMD:C_0603_1608Metric
- removed C55, C56, C58, C60, C63: 1uF, Capacitor_SMD:C_0603_1608Metric
- removed C57, C59, C64: 4.7uF, Capacitor_SMD:C_0603_1608Metric
- removed C62: 2.2nF, Capacitor_SMD:C_0603_1608Metric
- removed D3, D4: LED, LED_SMD:LED_0603_1608Metric
- removed J10: Prog, myLib:Pad_prog_4Pad
- removed J11: UART, myLib:Pad_3Pin_1.5x0.8mm
- removed J5: Touch Pads, myLib:Pad_3Pin_1.5x0.8mm
- removed J7: USB_C_Receptacle_USB2.0_16P, Connector_USB:USB_C_Receptacle_GCT_USB4110
- removed L10: 2.2uH, Inductor_SMD:L_0603_1608Metric
- removed L6: N.M., Inductor_SMD:L_0603_1608Metric
- removed L7: 2.2nH, Inductor_SMD:L_0603_1608Metric
- removed L8, L9: 10uH, Inductor_SMD:L_0603_1608Metric
- removed LS2, LS3: Boneconduction, myLib:Pad_2Pin_1.5x0.8mm
- removed LS6: SPH18R1LM4H-1-8, myLib:MIC_SPH18R1LM4H_KNO
- removed R13: 75k, Resistor_SMD:R_0603_1608Metric
- removed R20, R21, R27: 5K1R, Resistor_SMD:R_0603_1608Metric
- removed R26: 2R2, Resistor_SMD:R_0603_1608Metric
- removed R28: 10K, Resistor_SMD:R_0603_1608Metric
- removed R29, R30: 4k7, Resistor_SMD:R_0603_1608Metric
- removed R31, R32: 1K5R, Resistor_SMD:R_0603_1608Metric
- removed R33: 680k, Resistor_SMD:R_0603_1608Metric
- removed R7: N.C., Resistor_SMD:R_0603_1608Metric
- removed U10: NPM1100-CAAA-R7, myLib:NPM1100-CAAA-BGA25C40P5X5_207X207X52N
- removed U5: MAX98357AEWL_T, myLib:MAX98357A_BGA9N40P3X3_134X143X69N
- removed U7: MPR121QR2, myLib:MPR121
- removed U8: BMA400, myLib:QFN_BMA400_BOS
- removed U9: NRF5340-QKAA-R, Package_DFN_QFN:Nordic_AQFN-94-1EP_7x7mm_P0.4mm
- removed Y3: 32MHz, myLib:ECS-160-10-37-JTN-TR_ECS
- removed Y4: 32.768kHz, myLib:Crystal_24MHz-ECS-240-12-37B-CKY-TR
- Y2: footprint myLib:Crystal_24MHz-ECS-240-12-37B-CKY-TR -> lib:XTAL_ABS05-32.768KHZ-T
- moved R14 487.1 mm to (-17.4, -33.7)
- moved R15 487.1 mm to (-13.3, -48.8)
- moved R16 487.1 mm to (-13.3, -61.3)
- moved R17 487.1 mm to (-13.3, -43.8)
- moved R18 487.1 mm to (-13.3, -56.3)
- moved R19 487.1 mm to (-13.3, -53.8)
- moved R22 487.1 mm to (-17.4, -31.2)
- moved R23 487.1 mm to (-13.3, -46.3)
- moved R24 487.1 mm to (-13.3, -58.8)
- moved R25 487.1 mm to (-13.3, -41.2)
- moved C42 487.1 mm to (-33.4, -46.3)
- moved C45 487.1 mm to (-33.4, -31.2)
- moved C49 487.1 mm to (-33.4, -33.7)
- moved C50 487.1 mm to (-33.4, -43.8)
- moved C51 487.1 mm to (-29.4, -61.3)
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Connections:
- BT1 pad 2: (no net) -> GND
- BT1 pad 3: GND -> (no net)
- U3 pad A25: (no net) -> GND
- U3 pad AA1: (no net) -> GND
- U3 pad AE1: (no net) -> unconnected-(U3C-P1.02/TWI-PadAE1)
- U3 pad AE31: (no net) -> unconnected-(U3B-P0.28/AIN7-PadAE31)
- U3 pad AF2: (no net) -> unconnected-(U3C-P1.03/TWI-PadAF2)
- U3 pad AG31: (no net) -> unconnected-(U3A-DECF-PadAG31)
- U3 pad AH2: (no net) -> unconnected-(U3B-P0.08/TRACEDATA3/SCK-PadAH2)
- U3 pad AJ1: (no net) -> unconnected-(U3B-P0.09/TRACEDATA2/MOSI-PadAJ1)
- U3 pad AK10: (no net) -> unconnected-(U3B-P0.15/IO2-PadAK10)
- U3 pad AK12: (no net) -> unconnected-(U3B-P0.17/SCK-PadAK12)
- U3 pad AK14: (no net) -> unconnected-(U3B-P0.18/CSN-PadAK14)
- U3 pad AK16: (no net) -> /SD_MODE
- U3 pad AK18: (no net) -> /ISET
- U3 pad AK2: (no net) -> unconnected-(U3B-P0.10/TRACEDATA1/MISO-PadAK2)
- U3 pad AK20: (no net) -> unconnected-(U3B-P0.23-PadAK20)
- U3 pad AK22: (no net) -> unconnected-(U3C-P1.05-PadAK22)
- U3 pad AK24: (no net) -> unconnected-(U3C-P1.07-PadAK24)
- U3 pad AK26: (no net) -> unconnected-(U3C-P1.09-PadAK26)
- U3 pad AK28: (no net) -> /MIC_DATA
- U3 pad AK30: (no net) -> unconnected-(U3B-P0.27/AIN6-PadAK30)
- U3 pad AK4: (no net) -> unconnected-(U3B-P0.11/TRACEDATA0/CSN-PadAK4)
- U3 pad AK6: (no net) -> unconnected-(U3B-P0.12/TRACECLK/DCX-PadAK6)
- U3 pad AK8: (no net) -> unconnected-(U3B-P0.14/IO1-PadAK8)
- U3 pad AL13: (no net) -> unconnected-(U3B-P0.19-PadAL13)
- U3 pad AL15: (no net) -> /IRQ
- U3 pad AL19: (no net) -> unconnected-(U3C-P1.04-PadAL19)
- U3 pad AL21: (no net) -> unconnected-(U3C-P1.06-PadAL21)
- U3 pad AL23: (no net) -> unconnected-(U3C-P1.08-PadAL23)
- U3 pad AL27: (no net) -> unconnected-(U3B-P0.24-PadAL27)
- U3 pad AL29: (no net) -> /MIC_CLOCK
- U3 pad AL5: (no net) -> unconnected-(U3B-P0.13/IO0-PadAL5)
- U3 pad AL9: (no net) -> unconnected-(U3B-P0.16/IO3-PadAL9)
- U3 pad B14: (no net) -> unconnected-(U3C-P1.15-PadB14)
- U3 pad B20: (no net) -> unconnected-(U3C-P1.11-PadB20)
- U3 pad B22: (no net) -> unconnected-(U3B-P0.31-PadB22)
- U3 pad B24: (no net) -> unconnected-(U3B-P0.30-PadB24)
- U3 pad B26: (no net) -> GND
- U3 pad EP: (no net) -> GND
- U3 pad G1: (no net) -> GND
- U3 pad J1: (no net) -> unconnected-(U3A-DCCH-PadJ1)
- U3 pad J31: (no net) -> GND
- U3 pad R31: (no net) -> unconnected-(U3C-P1.10-PadR31)
- U3 pad T2: (no net) -> unconnected-(U3D-NC-PadT2)
- U3 pad U31: (no net) -> unconnected-(U3B-P0.29-PadU31)
- U3 pad W1: (no net) -> GND
Routing:
- net VDD: track 0.00 -> 148.7 mm, vias 0 -> 14
- net /LRCLK: track 0.00 -> 17.9 mm, vias 0 -> 2
- net Net-(U3A-DECN): track 0.00 -> 11.6 mm, vias 0 -> 2
- net Net-(U3A-VBUS): track 0.00 -> 11.2 mm, vias 0 -> 2
- net Net-(U3A-DECR): track 0.00 -> 10.2 mm, vias 0 -> 3
- net Net-(U3A-DCCD): track 0.00 -> 9.13 mm, vias 0 -> 2
- net Net-(U3A-DECD): track 0.00 -> 8.38 mm, vias 0 -> 2
- net Net-(U3D-XC1): track 0.00 -> 6.50 mm
- net Net-(U3D-XC2): track 0.00 -> 6.25 mm
- net Net-(U3A-DECUSB): track 0.00 -> 3.06 mm
- net GND: track 0.00 -> 2.94 mm, vias 0 -> 12
- net Net-(U3B-P0.01/XL2): track 0.00 -> 2.77 mm
- net Net-(U3B-P0.00/XL1): track 0.00 -> 2.51 mm
- net Net-(U3A-DECA): track 0.00 -> 2.48 mm
- net /D+: track 0.00 -> 0.64 mm, vias 0 -> 1
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- added copper zone on In1.Cu, net GND
Other:
- outline, holes or cut-outs redrawn
- copper layers 6 -> 4

Commit message: final, next is to order
Parts:
- added ?: , , B.Cu at (94.5, 93.4)
- added ?: , , B.Cu at (98.4, 93.4)
- added ?: , , B.Cu at (155.8, 93.4)
- added ?: , , B.Cu at (151.8, 93.4)
- added AE1: Antenna_Shield, RF_Antenna:Texas_SWRA117D_2.4GHz_Left, F.Cu at (168.4, 59.2)
- added BT1: Battery_Cell, myLib:Pad_3Pin_1.5x0.8mm, F.Cu at (162.4, 85.2)
- added C1: 100nF, Capacitor_SMD:C_0603_1608Metric, F.Cu at (140.9, 67.8)
- added C10: 100nF, Capacitor_SMD:C_0603_1608Metric, F.Cu at (138.8, 63.1)
- added C11: 100nF, Capacitor_SMD:C_0603_1608Metric, F.Cu at (139.3, 79.6)
- added C12: 1uF, Capacitor_SMD:C_0603_1608Metric, F.Cu at (158.5, 66.7)
- added C13: 1uF, Capacitor_SMD:C_0603_1608Metric, F.Cu at (167.0, 68.8)
- added C14: 4.7uF, Capacitor_SMD:C_0603_1608Metric, F.Cu at (153.5, 63.0)
- added C15: 1uF, Capacitor_SMD:C_0603_1608Metric, F.Cu at (153.6, 66.6)
- added C16: 4.7uF, Capacitor_SMD:C_0603_1608Metric, F.Cu at (155.2, 66.7)
- added C17: 1uF, Capacitor_SMD:C_0603_1608Metric, F.Cu at (157.5, 63.8)
- added C18: 100nF, Capacitor_SMD:C_0603_1608Metric, F.Cu at (155.1, 63.0)
- added C19: 2.2nF, Capacitor_SMD:C_0603_1608Metric, F.Cu at (164.4, 71.2)
- added C2: 0.1uF, Capacitor_SMD:C_0603_1608Metric, F.Cu at (139.3, 83.0)
- added C20: 1uF, Capacitor_SMD:C_0603_1608Metric, F.Cu at (156.9, 66.7)
- added C21: 4.7uF, Capacitor_SMD:C_0603_1608Metric, F.Cu at (147.2, 54.9)
- added C23: 0.1uF, Capacitor_SMD:C_0603_1608Metric, F.Cu at (174.3, 66.8)
- added C25: 10uF, Capacitor_SMD:C_0603_1608Metric, F.Cu at (174.3, 65.0)
- added C26: 10uF, Capacitor_SMD:C_0603_1608Metric, F.Cu at (148.8, 54.9)
- added C27: 10uF, Capacitor_SMD:C_0603_1608Metric, F.Cu at (147.6, 63.1)
- added C28: 10uF, Capacitor_SMD:C_0603_1608Metric, F.Cu at (150.5, 54.9)
- added C3: N.M., Capacitor_SMD:C_0603_1608Metric, F.Cu at (166.9, 77.4)
- added C30: 100nF, Capacitor_SMD:C_0603_1608Metric, F.Cu at (164.4, 73.0)
- added C31: 100nF, Capacitor_SMD:C_0603_1608Metric, F.Cu at (163.0, 77.1)
- added C32: 47uF, Capacitor_SMD:C_0603_1608Metric, F.Cu at (174.3, 63.0)
- added C33: 100nF, Capacitor_SMD:C_0603_1608Metric, F.Cu at (151.1, 69.7)
- added C34: 100nF, Capacitor_SMD:C_0603_1608Metric, F.Cu at (156.2, 79.6)
- added C35: 100nF, Capacitor_SMD:C_0603_1608Metric, F.Cu at (151.1, 76.9)
- added C36: 100nF, Capacitor_SMD:C_0603_1608Metric, F.Cu at (157.9, 79.6)
- added C37: 100nF, Capacitor_SMD:C_0603_1608Metric, F.Cu at (151.1, 75.2)
- added C38: 100nF, Capacitor_SMD:C_0603_1608Metric, F.Cu at (159.9, 62.3)
- added C4: N.M., Capacitor_SMD:C_0603_1608Metric, F.Cu at (170.6, 62.1)
- added C5: N.M., Capacitor_SMD:C_0603_1608Metric, F.Cu at (170.6, 60.5)
- added C6: 0.7pF, Capacitor_SMD:C_0603_1608Metric, F.Cu at (165.1, 77.4)
- added C7: 12pF, Capacitor_SMD:C_0603_1608Metric, F.Cu at (162.3, 64.2)
- added C8: 12pF, Capacitor_SMD:C_0603_1608Metric, F.Cu at (166.0, 66.0)
- added C9: 0.1uF, Capacitor_SMD:C_0603_1608Metric, F.Cu at (152.9, 81.2)
- added D1: LED, LED_SMD:LED_0603_1608Metric, F.Cu at (143.3, 61.3)
- added D2: LED, LED_SMD:LED_0603_1608Metric, F.Cu at (141.5, 61.3)
- added J1: USB_C_Receptacle_USB2.0_16P, Connector_USB:USB_C_Receptacle_GCT_USB4110, F.Cu at (131.4, 72.0)
- added J2: Touch Pads, myLib:Pad_3Pin_1.5x0.8mm, F.Cu at (147.1, 85.2)
- added J3: UART, myLib:Pad_3Pin_1.5x0.8mm, F.Cu at (155.3, 85.2)
- added J4: Prog, myLib:Pad_prog_4Pad, F.Cu at (170.3, 85.2)
- added L1: N.M., Inductor_SMD:L_0603_1608Metric, F.Cu at (168.3, 61.3)
- added L2: 2.2nH, Inductor_SMD:L_0603_1608Metric, F.Cu at (165.8, 75.0)
- added L3: 10uH, Inductor_SMD:L_0603_1608Metric, F.Cu at (165.1, 68.8)
- added L4: 10uH, Inductor_SMD:L_0603_1608Metric, F.Cu at (157.5, 62.2)
- added L5: 2.2uH, Inductor_SMD:L_0603_1608Metric, F.Cu at (150.0, 62.3)
- added LS1: SPH18R1LM4H-1-8, myLib:MIC_SPH18R1LM4H_KNO, F.Cu at (149.9, 80.8)
- added LS4: Boneconduction, myLib:Pad_2Pin_1.5x0.8mm, F.Cu at (174.2, 76.1)
- added LS5: Boneconduction, myLib:Pad_2Pin_1.5x0.8mm, F.Cu at (174.2, 78.5)
- added R1: 75k, Resistor_SMD:R_0603_1608Metric, F.Cu at (141.9, 84.6)
- added R10: 4k7, Resistor_SMD:R_0603_1608Metric, F.Cu at (145.6, 68.2)
- added R11: 1K5R, Resistor_SMD:R_0603_1608Metric, F.Cu at (141.5, 58.2)
- added R12: 1K5R, Resistor_SMD:R_0603_1608Metric, F.Cu at (143.3, 58.2)
- added R2: 5K1R, Resistor_SMD:R_0603_1608Metric, F.Cu at (138.7, 70.1)
- added R3: 5K1R, Resistor_SMD:R_0603_1608Metric, F.Cu at (138.8, 74.3)
- added R34: 680k, Resistor_SMD:R_0603_1608Metric, F.Cu at (171.2, 68.9)
- added R4: 2R2, Resistor_SMD:R_0603_1608Metric, F.Cu at (153.5, 60.0)
- added R5: 5K1R, Resistor_SMD:R_0603_1608Metric, F.Cu at (144.0, 54.9)
- added R6: 10K, Resistor_SMD:R_0603_1608Metric, F.Cu at (145.6, 54.9)
- added R8: N.C., Resistor_SMD:R_0603_1608Metric, F.Cu at (174.2, 72.5)
- added R9: 4k7, Resistor_SMD:R_0603_1608Metric, F.Cu at (145.6, 66.4)
- added REF**: Pad_1Pin_2x1.2mm, myLib:Pad_1Pin_2x1.2mm, B.Cu at (96.4, 93.4)
- added REF**: Pad_1Pin_2x1.2mm, myLib:Pad_1Pin_2x1.2mm, B.Cu at (153.8, 93.4)
- added U1: BMA400, myLib:QFN_BMA400_BOS, F.Cu at (141.4, 65.0)
- added U2: MPR121QR2, myLib:MPR121, F.Cu at (143.2, 81.3)
- added U3: NRF5340-QKAA-R, Package_DFN_QFN:Nordic_AQFN-94-1EP_7x7mm_P0.4mm, F.Cu at (157.5, 73.1)
- added U4: NPM1100-CAAA-R7, myLib:NPM1100-CAAA-BGA25C40P5X5_207X207X52N, F.Cu at (147.0, 59.8)
- added U6: MAX98357AEWL_T, myLib:MAX98357A_BGA9N40P3X3_134X143X69N, F.Cu at (174.3, 69.8)
- added Y1: 32MHz, myLib:YSX321SL - 32Mhz Crystal, F.Cu at (161.8, 66.9)
- added Y2: 32.768kHz, lib:XTAL_ABS05-32.768KHZ-T, F.Cu at (151.8, 73.0)
- Y1: footprint myLib:ECS-160-10-37-JTN-TR_ECS -> myLib:YSX321SL - 32Mhz Crystal
- moved J9 232.2 mm to (133.5, 91.6)
- moved C51 223.3 mm to (124.3, 100.7), turned to -90 degrees
- moved J8 221.1 mm to (130.0, 97.3)
- moved J6 212.0 mm to (114.7, 97.3)
- moved C42 211.0 mm to (117.9, 100.7), turned to -90 degrees
- moved R16 210.8 mm to (120.5, 101.6)
- moved C50 208.0 mm to (120.6, 96.0)
- moved R24 207.2 mm to (122.3, 97.8), turned to 180 degrees
- moved R23 202.4 mm to (126.8, 99.8)
- moved C45 201.7 mm to (124.4, 94.5), turned to -90 degrees
- moved R25 200.1 mm to (126.8, 101.6)
- moved R15 199.8 mm to (126.8, 93.6)
- moved R19 199.3 mm to (121.1, 93.3), turned to 90 degrees
- moved R18 198.9 mm to (118.7, 92.4)
- moved C49 198.7 mm to (118.7, 94.2)
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Routing:
- net GND: track 2.94 -> 228.6 mm, vias 12 -> 110
- net VDD: track 148.7 -> 353.4 mm, vias 14 -> 52
- net +3.3V: track 0.00 -> 143.2 mm, vias 0 -> 12
- net /D+: track 0.64 -> 84.4 mm, vias 1 -> 8
- net /D-: track 0.00 -> 82.2 mm, vias 1 -> 6
- net VBUS: track 0.00 -> 78.1 mm, vias 0 -> 10
- net /I2C_SCL: track 0.00 -> 68.5 mm, vias 1 -> 10
- net /I2C_SDA: track 0.00 -> 64.2 mm, vias 1 -> 12
- net /IRQ: track 0.00 -> 53.7 mm, vias 0 -> 4
- net /SD_MODE: track 0.00 -> 42.7 mm, vias 0 -> 4
- net /ISET: track 0.00 -> 42.0 mm, vias 0 -> 4
- net /INT2: track 0.00 -> 40.1 mm, vias 1 -> 6
- net /INT1: track 0.00 -> 37.6 mm, vias 1 -> 6
- net /SDOUT: track 0.00 -> 37.4 mm, vias 0 -> 4
- net /MIC_DATA: track 0.00 -> 36.1 mm, vias 0 -> 4
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- added copper zone on F.Cu, net Net-(J2-Pin_1)
- added copper zone on F.Cu, net Net-(J2-Pin_2)
- added copper zone on F.Cu, net Net-(J2-Pin_3)
Other:
- board size 49.3 x 34.5 mm -> 105.2 x 51.3 mm
- board text added: "+"
- board text added: "-"
- board text added: "->"
- board text added: "1"
- board text added: "BAT"
- board text added: "HIGH V"
- board text added: "LOW V"
- board text added: "Logic Level Shifter Programer"
- board text added: "MSBE Left 0100 1101"
- board text added: "MSBE Right 0100 1101"
- board text added: "Prog"
- board text added: "Touch Pads"
