File: hardware/kicad/ver_1.0/MSBE_V3.kicad_pcb (KiCad board)
At the start: 4 copper layers, 105.2 x 51.3 mm, 164 parts, among them J1 USB_C_Receptacle_USB2.0_16P, J2 Touch Pads, J3 UART, J4 Prog, J6 High-V, J8 Low-V, J9 Low-V-TH, U1 BMA400, U2 MPR121QR2, U3 NRF5340-QKAA-R, U4 NPM1100-CAAA-R7, U6 MAX98357AEWL_T, Y1 32MHz, Y2 32.768kHz

Commit message: newest BGA started
Parts:
- removed ? (x4): , 
- removed the AE1 at (168.4, 59.2)
- removed the BT1 at (162.4, 85.2)
- removed the C1 at (140.9, 67.8)
- removed the C10 at (138.8, 63.1)
- removed the C11 at (139.3, 79.6)
- removed the C12 at (158.5, 66.7)
- removed the C13 at (167.0, 68.8)
- removed the C14 at (153.5, 63.0)
- removed the C15 at (153.6, 66.6)
- removed the C16 at (155.2, 66.7)
- removed the C17 at (157.5, 63.8)
- removed the C18 at (155.1, 63.0)
- removed the C19 at (164.4, 71.2)
- removed the C2 at (139.3, 83.0)
- removed the C20 at (156.9, 66.7)
- removed the C21 at (147.2, 54.9)
- removed the C23 at (174.3, 66.8)
- removed the C25 at (174.3, 65.0)
- removed the C26 at (148.8, 54.9)
- removed the C27 at (147.6, 63.1)
- removed the C28 at (150.5, 54.9)
- removed the C3 at (166.9, 77.4)
- removed the C30 at (164.4, 73.0)
- removed the C31 at (163.0, 77.1)
- removed the C32 at (174.3, 63.0)
- removed the C33 at (151.1, 69.7)
- removed the C34 at (156.2, 79.6)
- removed the C35 at (151.1, 76.9)
- removed the C36 at (157.9, 79.6)
- removed the C37 at (151.1, 75.2)
- removed the C38 at (159.9, 62.3)
- removed the C4 at (170.6, 62.1)
- removed the C5 at (170.6, 60.5)
- removed the C6 at (165.1, 77.4)
- removed the C7 at (162.3, 64.2)
- removed the C8 at (166.0, 66.0)
- removed the C9 at (152.9, 81.2)
- removed the D1 at (143.3, 61.3)
- removed the D2 at (141.5, 61.3)
- removed the J1 at (131.4, 72.0)
- removed the J2 at (147.1, 85.2)
- removed the J3 at (155.3, 85.2)
- removed the J4 at (170.3, 85.2)
- removed the L1 at (168.3, 61.3)
- removed the L2 at (165.8, 75.0)
- removed the L3 at (165.1, 68.8)
- removed the L4 at (157.5, 62.2)
- removed the L5 at (150.0, 62.3)
- removed the LS1 at (149.9, 80.8)
- removed the LS4 at (174.2, 76.1)
- removed the LS5 at (174.2, 78.5)
- removed the R1 at (141.9, 84.6)
- removed the R10 at (145.6, 68.2)
- removed the R11 at (141.5, 58.2)
- removed the R12 at (143.3, 58.2)
- removed the R2 at (138.7, 70.1)
- removed the R3 at (138.8, 74.3)
- removed the R34 at (171.2, 68.9)
- removed the R4 at (153.5, 60.0)
- removed the R5 at (144.0, 54.9)
- removed the R6 at (145.6, 54.9)
- removed the R8 at (174.2, 72.5)
- removed the R9 at (145.6, 66.4)
- removed REF** (x2): Pad_1Pin_2x1.2mm, myLib:Pad_1Pin_2x1.2mm
- removed the U1 at (141.4, 65.0)
- removed the U2 at (143.2, 81.3)
- removed the U3 at (157.5, 73.1)
- removed the U4 at (147.0, 59.8)
- removed the U6 at (174.3, 69.8)
- removed the Y1 at (161.8, 66.9)
- removed the Y2 at (151.8, 73.0)
- U6: footprint myLib:MAX98357A_BGA9N40P3X3_134X143X69N -> lib:MAX98357AETE_QFN16
- moved J9 50.3 mm to (86.9, 110.6), turned to 180 degrees
- moved J8 40.2 mm to (90.5, 104.9), turned to 180 degrees
- moved R15 36.4 mm to (93.6, 108.6), turned to 180 degrees
- moved R17 35.1 mm to (93.6, 106.8), turned to 180 degrees
- moved R23 33.2 mm to (93.7, 102.4), turned to 180 degrees
- moved R25 33.1 mm to (93.7, 100.6), turned to 180 degrees
- moved C45 31.3 mm to (96.0, 107.7), turned to 90 degrees
- moved C51 28.2 mm to (96.1, 101.5), turned to 90 degrees
- moved R19 26.8 mm to (99.3, 108.8), turned to -90 degrees
- moved R24 25.1 mm to (98.1, 104.4), turned to 0 degrees
- moved R18 24.2 mm to (101.8, 109.7), turned to 180 degrees
- moved C50 23.0 mm to (99.9, 106.1), turned to 180 degrees
- moved C49 21.8 mm to (101.8, 108.0), turned to 180 degrees
- moved R14 20.7 mm to (100.0, 102.3), turned to 180 degrees
- moved R16 20.5 mm to (100.0, 100.6), turned to 180 degrees
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Connections:
- C1 pad 1: VDD -> +3.3V
- C10 pad 2: VDD -> +3.3V
- C11 pad 1: VDD -> +3.3V
- C12 pad 1: VDD -> +3.3V
- C15 pad 1: VDD -> +3.3V
- C27 pad 2: VDD -> +3.3V
- C30 pad 1: VDD -> +3.3V
- C31 pad 1: VDD -> +3.3V
- C33 pad 1: VDD -> +3.3V
- C34 pad 1: VDD -> +3.3V
- C35 pad 1: VDD -> +3.3V
- C36 pad 1: VDD -> +3.3V
- C37 pad 1: VDD -> +3.3V
- C38 pad 1: VDD -> +3.3V
- C9 pad 1: VDD -> +3.3V
- J4 pad 1: VDD -> +3.3V
- L5 pad 1: VDD -> +3.3V
- LS1 pad 5: VDD -> +3.3V
- R10 pad 2: VDD -> +3.3V
- R34 pad 1: VDD -> +3.3V
- R9 pad 2: VDD -> +3.3V
- U1 pad 10: VDD -> +3.3V
- U1 pad 3: VDD -> +3.3V
- U1 pad 7: VDD -> +3.3V
- U2 pad 20: VDD -> +3.3V
- U3 pad A19: VDD -> +3.3V
- U3 pad AC1: VDD -> +3.3V
- U3 pad AG1: VDD -> +3.3V
- U3 pad AJ31: VDD -> +3.3V
- U3 pad AL11: VDD -> +3.3V
- U3 pad AL17: VDD -> +3.3V
- U3 pad AL25: VDD -> +3.3V
- U3 pad AL3: VDD -> +3.3V
- U3 pad AL7: VDD -> +3.3V
- U3 pad B28: VDD -> +3.3V
- U3 pad B8: VDD -> +3.3V
- U3 pad C1: VDD -> +3.3V
- U3 pad E1: VDD -> +3.3V
- U3 pad E31: VDD -> +3.3V
- U3 pad EP: GND -> (no net)
- U3 pad L1: VDD -> +3.3V
- U3 pad N31: VDD -> +3.3V
- U3 pad U1: VDD -> +3.3V
- U4 pad B5: VDD -> +3.3V
- U4 pad C3: VDD -> +3.3V
- Y1 pad 4: GND -> (no net)
Routing:
- net VDD: track 353.4 -> 0.00 mm, vias 52 -> 0
- net GND: track 228.6 -> 104.9 mm, vias 110 -> 52
- net +3.3V: track 143.2 -> 239.7 mm, vias 12 -> 30
- net /D+: track 84.4 -> 42.2 mm, vias 8 -> 4
- net /D-: track 82.2 -> 41.1 mm, vias 6 -> 3
- net VBUS: track 78.1 -> 39.1 mm, vias 10 -> 5
- net /I2C_SCL: track 68.5 -> 34.2 mm, vias 10 -> 5
- net /I2C_SDA: track 64.2 -> 32.1 mm, vias 12 -> 6
- net /IRQ: track 53.7 -> 26.8 mm, vias 4 -> 2
- net /SD_MODE: track 42.7 -> 16.1 mm, vias 4 -> 1
- net /LRCLK: track 37.0 -> 15.9 mm, vias 4 -> 1
- net /ISET: track 42.0 -> 21.0 mm, vias 4 -> 2
- net /INT2: track 40.1 -> 20.1 mm, vias 6 -> 3
- net /SDOUT: track 37.4 -> 17.8 mm, vias 4 -> 1
- net /INT1: track 37.6 -> 18.8 mm, vias 6 -> 3
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Other:
- board size 105.2 x 51.3 mm -> 49.3 x 60.1 mm
- board text added: "MSBE 0100 1101"
- board text removed: "MSBE Left 0100 1101"
- board text removed: "MSBE Right 0100 1101"
- board text removed: "Touch Pads"
