File: hardware/kicad/ver_1.0/MSBE_V3.kicad_sch (KiCad schematic)
At the start: 156 parts, among them J1 USB_C_Receptacle_USB2.0_16P, J10 Prog, J11 UART, J2 Touch Pads, J3 UART, J4 Prog, J5 Touch Pads, J6 High-V, J7 USB_C_Receptacle_USB2.0_16P, J8 Low-V, J9 Low-V-TH, U1 BMA400, U10 NPM1100-CAAA-R7, U2 MPR121QR2, U3 NRF5340-QKAA-R, U4 NPM1100-CAAA-R7, U5 MAX98357AEWL_T, U6 MAX98357AEWL_T, U7 MPR121QR2, U8 BMA400, U9 NRF5340-QKAA-R, Y1 32MHz, Y2 32.768kHz, Y3 32MHz, Y4 32.768kHz

Commit message: izmena
Parts:
- added R33, R34: 680k, Resistor_SMD:R_0603_1608Metric, symbol Device:R
Connections:
- net SD_MODE: now also R33.2, R34.2
- net VDD: now also R33.1, R34.1
Other:
- note added: "High-impedance input"
- note added: "ON - MCU SD pin input (High impedance) OFF - MCU SD pin output (LOW)"
