File: hardware/kicad/ver_1.0/MSBE_V3.kicad_sch (KiCad schematic)
At the start: 158 parts, among them J1 USB_C_Receptacle_USB2.0_16P, J10 Prog, J11 UART, J2 Touch Pads, J3 UART, J4 Prog, J5 Touch Pads, J6 High-V, J7 USB_C_Receptacle_USB2.0_16P, J8 Low-V, J9 Low-V-TH, U1 BMA400, U10 NPM1100-CAAA-R7, U2 MPR121QR2, U3 NRF5340-QKAA-R, U4 NPM1100-CAAA-R7, U5 MAX98357AEWL_T, U6 MAX98357AEWL_T, U7 MPR121QR2, U8 BMA400, U9 NRF5340-QKAA-R, Y1 32MHz, Y2 32.768kHz, Y3 32MHz, Y4 32.768kHz

Commit message: izmene 7.11
Connections:
- net IRQ: now also U3.AL15 (P0.21)
- net RX: now also U3.P2 (P1.01)
- net TX: now also U3.M2 (P1.00)
Other:
- note added: "Enable software pull-up"
Changed lines of the file:
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@@
 		)
 	)
+	(text "Enable software pull-up\n"
+		(exclude_from_sim no)
+		(at 178.562 236.982 0)
+		(effects
+			(font
+				(size 1.27 1.27)
+			)
+			(justify right)
+		)
+	)
 	(text "RIGHT CHANNEL SELECTED"
 		(exclude_from_sim no)
@@
 		)
 	)
+	(label "IRQ"
+		(at 179.07 237.49 0)
+		(effects
+			(font
+				(size 1.27 1.27)
+			)
+			(justify left bottom)
+		)
+	)
 	(label "MIC_CLOCK"
 		(at 179.07 250.19 0)
@@
 		)
 	)
+	(label "TX"
+		(at 118.11 92.71 180)
+		(effects
+			(font
+				(size 1.27 1.27)
+			)
+			(justify right bottom)
+		)
+	)
 	(label "MIC_CLOCK"
 		(at 496.57 257.81 0)
@@
 		)
 	)
+	(label "RX"
+		(at 118.11 90.17 180)
+		(effects
+			(font
+				(size 1.27 1.27)
+			)
+			(justify right bottom)
+		)
+	)

Commit message: start of routing
Parts:
- removed AE2: Antenna_Shield, RF_Antenna:Texas_SWRA117D_2.4GHz_Left, symbol Device:Antenna_Shield
- removed BT2: Battery_Cell, myLib:Pad_3Pin_1.5x0.8mm, symbol Device:Battery_Cell
- removed C22, C39, C53: 0.1uF, Capacitor_SMD:C_0603_1608Metric, symbol Device:C
- removed C24, C65, C66, C67: 10uF, Capacitor_SMD:C_0603_1608Metric, symbol Device:C
- removed C29: 47uF, Capacitor_SMD:C_0603_1608Metric, symbol Device:C
- removed C40, C52, C54, C61, C68, C69, C70, C71, C72, C73, C74, C75: 100nF, Capacitor_SMD:C_0603_1608Metric, symbol Device:C
- removed C41, C43, C44: N.M., Capacitor_SMD:C_0603_1608Metric, symbol Device:C
- removed C46: 0.7pF, Capacitor_SMD:C_0603_1608Metric, symbol Device:C
- removed C47, C48: 12pF, Capacitor_SMD:C_0603_1608Metric, symbol Device:C
- removed C55, C56, C58, C60, C63: 1uF, Capacitor_SMD:C_0603_1608Metric, symbol Device:C
- removed C57, C59, C64: 4.7uF, Capacitor_SMD:C_0603_1608Metric, symbol Device:C
- removed C62: 2.2nF, Capacitor_SMD:C_0603_1608Metric, symbol Device:C
- removed D3, D4: LED, LED_SMD:LED_0603_1608Metric, symbol Device:LED
- removed J10: Prog, myLib:Pad_prog_4Pad, symbol Connector:Conn_01x05_Pin
- removed J11: UART, myLib:Pad_3Pin_1.5x0.8mm, symbol Connector:Conn_01x03_Pin
- removed J5: Touch Pads, myLib:Pad_3Pin_1.5x0.8mm, symbol Connector:Conn_01x03_Pin
- removed J7: USB_C_Receptacle_USB2.0_16P, Connector_USB:USB_C_Receptacle_GCT_USB4110, symbol Connector:USB_C_Receptacle_USB2.0_16P
- removed L10: 2.2uH, Inductor_SMD:L_0603_1608Metric, symbol Device:L
- removed L6: N.M., Inductor_SMD:L_0603_1608Metric, symbol Device:L
- removed L7: 2.2nH, Inductor_SMD:L_0603_1608Metric, symbol Device:L
- removed L8, L9: 10uH, Inductor_SMD:L_0603_1608Metric, symbol Device:L
- removed LS2, LS3: Boneconduction, myLib:Pad_2Pin_1.5x0.8mm, symbol Device:Speaker
- removed LS6: SPH18R1LM4H-1-8, myLib:MIC_SPH18R1LM4H_KNO, symbol mySch_lib:SPH18R1LM4H-1-8
- removed R13: 75k, Resistor_SMD:R_0603_1608Metric, symbol Device:R
- removed R20, R21, R27: 5K1R, Resistor_SMD:R_0603_1608Metric, symbol Device:R
- removed R26: 2R2, Resistor_SMD:R_0603_1608Metric, symbol Device:R
- removed R28: 10K, Resistor_SMD:R_0603_1608Metric, symbol Device:R
- removed R29, R30: 4k7, Resistor_SMD:R_0603_1608Metric, symbol Device:R
- removed R31, R32: 1K5R, Resistor_SMD:R_0603_1608Metric, symbol Device:R
- removed R33: 680k, Resistor_SMD:R_0603_1608Metric, symbol Device:R
- removed R7: N.C., Resistor_SMD:R_0603_1608Metric, symbol Device:R
- removed U10: NPM1100-CAAA-R7, myLib:NPM1100-CAAA-BGA25C40P5X5_207X207X52N, symbol mySch_lib:NPM1100-CAAA-R7
- removed U5: MAX98357AEWL_T, myLib:MAX98357A_BGA9N40P3X3_134X143X69N, symbol mySch_lib:MAX98357AEWL_T
- removed U7: MPR121QR2, myLib:MPR121, symbol mySch_lib:MPR121QR2
- removed U8: BMA400, myLib:QFN_BMA400_BOS, symbol mySch_lib:BMA400
- removed U9: NRF5340-QKAA-R, myLib:NRF5340, symbol 1_MSBE_V3-altium-import:root_0_NRF5340-QKAA-R_
- removed Y3: 32MHz, myLib:ECS-160-10-37-JTN-TR_ECS, symbol Device:Crystal
- removed Y4: 32.768kHz, myLib:Crystal_24MHz-ECS-240-12-37B-CKY-TR, symbol Device:Crystal
Connections:
- no-connect marks 44 -> 22
Other:
- note removed: "LEFT CHANNEL SELECTED"
- note removed: "Right"

Commit message: newest BGA started
Parts:
- U6: symbol mySch_lib:MAX98357AEWL_T -> lib:MAX98357AETE_
Connections:
- net VDD is gone; now on net +3.3V: C1.1, C10.2, C11.1, C12.1, C15.1, C27.2, C30.1, C31.1, C33.1, C34.1, C35.1, C36.1, C37.1, C38.1, C9.1, J4.1 (Pin_1), L5.1, LS1.5 (VDD), R10.2, R34.1, R9.2, U1.10 (CSB), U1.3 (VDDIO), U1.7 (VDD), U2.20 (VDD), U3.A19 (VDD), U3.AC1 (VDD), U3.AG1 (VDD), U3.AJ31 (VDD), U3.AL11 (VDD), U3.AL17 (VDD), U3.AL25 (VDD), U3.AL3 (VDD), U3.AL7 (VDD), U3.B28 (VDD), U3.B8 (VDD), U3.C1 (VDD), U3.E1 (VDDH), U3.E31 (VDD), U3.L1 (VDD), U3.N31 (VDD), U3.U1 (VDD), U4.B5 (VOUTB), U4.C3 (VTERMSET)
- net +3.3V: now also U6.7 (VDD), U6.8 (VDD); no longer U6.A2 (VDD)
- net AVSS: now also U6.11 (GND), U6.15 (GND), U6.17 (EP), U6.3 (GND); no longer U6.C2 (GND)
- net LRCLK: now also U6.14 (LRCLK); no longer U6.C3 (LRCLK)
- net SCK: now also U6.16 (BCLK); no longer U6.C1 (BCLK)
- net SDOUT: now also U6.1 (DIN); no longer U6.B1 (DIN)
- net SD_MODE: now also U6.4 (~{SD_MODE}); no longer U6.A1 (SD_MODE)
- net at R8.2: now also U6.2 (GAIN_SLOT); no longer U6.B2 (GAIN_SLOT)
- net at LS4.1, LS5.1: now also U6.10 (OUTN); no longer U6.B3 (OUTN)
- net at LS4.2, LS5.2: now also U6.9 (OUTP); no longer U6.A3 (OUTP)
Other:
- moved on the sheet: C23, C25, C32, LS4, LS5, R34, R8
