File: hardware/kicad/ver_1.0/untitled.kicad_sch (KiCad schematic)
At the start: 88 parts, among them J10 Low-V, J11 USB_C_Receptacle_USB2.0_16P, J12 Touch Pads, J13 UART, J14 Prog, J9 High-V, U10 MAX98357AEWL_T, U11 NPM1100-CAAA-R7, U12 NRF5340-CLAA-R, U13 BMA400, U14 MPR121QR2, U9 MAX98357AEWL_T, Y3 Crystal

Commit message: izmene 7.11
Parts:
- removed BT3: Battery_Cell, myLib:Pad_2Pin_1.5x0.8mm, symbol Device:Battery_Cell
- removed C100, C80, C81, C84, C85, C93, C95, C96, C97, C99: 100nF, Capacitor_SMD:C_0603_1608Metric, symbol Device:C
- removed C101, C76, C98: 0.1uF, Capacitor_SMD:C_0603_1608Metric, symbol Device:C
- removed C72, C88, C90: 4.7uF, Capacitor_SMD:C_0603_1608Metric, symbol Device:C
- removed C73, C74, C75: 10uF, Capacitor_SMD:C_0603_1608Metric, symbol Device:C
- removed C77, C78: 12pF, Capacitor_SMD:C_0603_1608Metric, symbol Device:C
- removed C79, C82, C86, C87, C94: 1.0uF, Capacitor_SMD:C_0603_1608Metric, symbol Device:C
- removed C83: 2.2nF, Capacitor_SMD:C_0603_1608Metric, symbol Device:C
- removed C89, C91: N.C., Capacitor_SMD:C_0603_1608Metric, symbol Device:C
- removed C92: 0.7pF, Capacitor_SMD:C_0603_1608Metric, symbol Device:C
- removed D5, D6: LED, LED_SMD:LED_0603_1608Metric, symbol Device:LED
- removed J11: USB_C_Receptacle_USB2.0_16P, Connector_USB:USB_C_Receptacle_GCT_USB4110, symbol Connector:USB_C_Receptacle_USB2.0_16P
- removed J12: Touch Pads, myLib:Pad_1Pin_2x1.2mm, symbol Connector:Conn_01x03_Pin
- removed J13: UART, myLib:Pad_3Pin_1.5x0.8mm, symbol Connector:Conn_01x03_Pin
- removed J14: Prog, myLib:Pad_prog_4Pad, symbol Connector:Conn_01x05_Pin
- removed L10, L11: 10uH, Inductor_SMD:L_0603_1608Metric, symbol Device:L
- removed L12: 2.2nH, Inductor_SMD:L_0603_1608Metric, symbol Device:L
- removed L9: 2.2uH, Inductor_SMD:L_0603_1608Metric, symbol Device:L
- removed LS7: SPH18R1LM4H-1-8, myLib:MIC_SPH18R1LM4H_KNO, symbol mySch_lib:SPH18R1LM4H-1-8
- removed R35, R37, R38: 5K1R, Resistor_SMD:R_0603_1608Metric, symbol Device:R
- removed R36: 10K, Resistor_SMD:R_0603_1608Metric, symbol Device:R
- removed R39, R40: 4.7k, Resistor_SMD:R_0603_1608Metric, symbol Device:R
- removed R41: 2R2, Resistor_SMD:R_0603_1608Metric, symbol Device:R
- removed R42: 75k, Resistor_SMD:R_0603_1608Metric, symbol Device:R
- removed U11: NPM1100-CAAA-R7, myLib:NPM1100-CAAA-BGA25C40P5X5_207X207X52N, symbol mySch_lib:NPM1100-CAAA-R7
- removed U12: NRF5340-CLAA-R, myLib:NRF5340, symbol mySch_lib:NRF5340-CLAA-R
- removed U13: BMA400, myLib:QFN_BMA400_BOS, symbol mySch_lib:BMA400
- removed U14: MPR121QR2, myLib:MPR121, symbol mySch_lib:MPR121QR2
- removed Y3: Crystal, myLib:Crystal_24MHz-ECS-240-12-37B-CKY-TR, symbol Device:Crystal
- added AE1: Antenna_Shield, RF_Antenna:Texas_SWRA117D_2.4GHz_Left, symbol Device:Antenna_Shield
- added BT1: Battery_Cell, myLib:Pad_3Pin_1.5x0.8mm, symbol Device:Battery_Cell
- added C1, C10, C11, C18, C30, C31, C33, C34, C35, C36, C37, C38: 100nF, Capacitor_SMD:C_0603_1608Metric, symbol Device:C
- added C12, C13, C15, C17, C20: 1uF, Capacitor_SMD:C_0603_1608Metric, symbol Device:C
- added C14, C16, C21: 4.7uF, Capacitor_SMD:C_0603_1608Metric, symbol Device:C
- added C19: 2.2nF, Capacitor_SMD:C_0603_1608Metric, symbol Device:C
- added C2, C9: 0.1uF, Capacitor_SMD:C_0603_1608Metric, symbol Device:C
- added C26, C27, C28: 10uF, Capacitor_SMD:C_0603_1608Metric, symbol Device:C
- added C3, C4, C5: N.M., Capacitor_SMD:C_0603_1608Metric, symbol Device:C
- added C6: 0.7pF, Capacitor_SMD:C_0603_1608Metric, symbol Device:C
- added C7, C8: 12pF, Capacitor_SMD:C_0603_1608Metric, symbol Device:C
- added D1, D2: LED, LED_SMD:LED_0603_1608Metric, symbol Device:LED
- added J1: USB_C_Receptacle_USB2.0_16P, Connector_USB:USB_C_Receptacle_GCT_USB4110, symbol Connector:USB_C_Receptacle_USB2.0_16P
- added J2: Touch Pads, myLib:Pad_3Pin_1.5x0.8mm, symbol Connector:Conn_01x03_Pin
- added J3: UART, myLib:Pad_3Pin_1.5x0.8mm, symbol Connector:Conn_01x03_Pin
- added J4: Prog, myLib:Pad_prog_4Pad, symbol Connector:Conn_01x05_Pin
- added J9: Low-V-TH, Connector_PinHeader_2.54mm:PinHeader_1x05_P2.54mm_Vertical, symbol Connector:Conn_01x05_Pin
- added L1: N.M., Inductor_SMD:L_0603_1608Metric, symbol Device:L
- added L2: 2.2nH, Inductor_SMD:L_0603_1608Metric, symbol Device:L
- added L3, L4: 10uH, Inductor_SMD:L_0603_1608Metric, symbol Device:L
- added L5: 2.2uH, Inductor_SMD:L_0603_1608Metric, symbol Device:L
- added LS1: SPH18R1LM4H-1-8, myLib:MIC_SPH18R1LM4H_KNO, symbol mySch_lib:SPH18R1LM4H-1-8
- added R1: 75k, Resistor_SMD:R_0603_1608Metric, symbol Device:R
- added R10, R9: 4k7, Resistor_SMD:R_0603_1608Metric, symbol Device:R
- added R11, R12: 1K5R, Resistor_SMD:R_0603_1608Metric, symbol Device:R
- added R2, R3, R5: 5K1R, Resistor_SMD:R_0603_1608Metric, symbol Device:R
- added R4: 2R2, Resistor_SMD:R_0603_1608Metric, symbol Device:R
- added R6: 10K, Resistor_SMD:R_0603_1608Metric, symbol Device:R
- added U1: BMA400, myLib:QFN_BMA400_BOS, symbol mySch_lib:BMA400
- added U2: MPR121QR2, myLib:MPR121, symbol mySch_lib:MPR121QR2
- added U3: NRF5340-QKAA-R, myLib:NRF5340, symbol 1_MSBE_V3-altium-import:root_0_NRF5340-QKAA-R_
- added U4: NPM1100-CAAA-R7, myLib:NPM1100-CAAA-BGA25C40P5X5_207X207X52N, symbol mySch_lib:NPM1100-CAAA-R7
- added Y1: 32MHz, myLib:ECS-160-10-37-JTN-TR_ECS, symbol Device:Crystal
- added Y2: 32.768kHz, myLib:Crystal_24MHz-ECS-240-12-37B-CKY-TR, symbol Device:Crystal
- R33, R34: value 1K5R -> 680k
- renumbered C63 to C22, C69 to C23, C64 to C24, C70 to C25, C65 to C29, C71 to C32, C61 to C42, C67 to C45, C66 to C49, C62 to C50, C68 to C51, J9 to J6, J10 to J8, LS3 to LS2, LS4 to LS3, LS5 to LS4, LS6 to LS5, R21 to R14, R28 to R15, R23 to R16, R30 to R17, R25 to R18, R26 to R19, R29 to R23, R31 to R25, R27 to R7, R32 to R8, U9 to U5, U10 to U6
Connections:
- net +3.3V: now also BT1.1 (+), C21.2, U4.D1 (VBAT), U4.D2 (VBAT)
- net AVSS: now also AE1.2 (Shield), BT1.2 (-), C1.2, C10.1, C11.2, C12.2, C13.2, C14.2, C15.2, C16.2, C17.2, C18.2, C19.2, C2.2, C20.2, C21.1, C26.1, C27.1, C28.1, C3.2, C30.2, C31.2, C33.2, C34.2, C35.2, C36.2, C37.2, C38.2, C4.2, C5.2, C6.2, C7.2, C8.2, C9.2, J1.A1 (GND), J1.A12 (GND), J1.B1 (GND), J1.B12 (GND), J1.S1 (SHIELD), J3.3 (Pin_3), J4.4 (Pin_4), LS1.3 (GROUND), R1.2, R2.1, R3.1, R5.1, R6.1, U1.1 (SDO), U1.8 (GNDIO), U1.9 (GND), U2.4 (ADDR), U2.6 (VSS), U3.104 (VSS), U3.A25 (VSS), U3.AA1 (P0.03/NFC2), U3.B12 (VSS), U3.B26 (VSS), U3.G1 (VSS), U3.H2 (VSS), U3.J31 (VSS), U3.W1 (P0.02/NFC1), U4.A5 (PVSS), U4.B3 (VOUTBSET1), U4.B4 (VOUTBSET0), U4.C4 (AVSS), U4.C5 (AVSS), U4.D3 (SHPHLD), U4.D4 (SHPACT), U4.E5 (MODE)
- net B1: now also J9.5 (Pin_5)
- net B2: now also J9.4 (Pin_4)
- net B3: now also J9.3 (Pin_3)
- net B4: now also J9.2 (Pin_2)
- net B5: now also J9.1 (Pin_1)
- net D+: now also J1.A6 (D+), J1.B6 (D+), U3.B2 (D+), U4.A2 (D+)
- net D-: now also J1.A7 (D-), J1.B7 (D-), U3.B4 (D-), U4.A1 (D-)
- net I2C_SCL: now also R9.1, U1.12 (SCX), U2.2 (SCL), U3.V2 (P0.04/AIN0)
- net I2C_SDA: now also R10.1, U1.2 (SDX), U2.3 (SDA), U3.Y2 (P0.05/AIN1)
- net INT1: now also U1.5 (INT1), U3.AB2 (P0.06/AIN2)
- net INT2: now also U1.6 (INT2), U3.AD2 (P0.07/AIN3)
- net IRQ: now also U2.1 (*IRQ)
- net ISET: now also U3.AK18 (P0.22), U4.D5 (ISET)
- net LRCLK: now also U3.A17 (P1.13)
- net MIC_CLOCK: now also LS1.4 (CLOCK), U3.AL29 (P0.26/AIN5)
- net MIC_DATA: now also LS1.1 (DATA), U3.AK28 (P0.25/AIN4)
- net RX: now also J3.2 (Pin_2)
- net SCK: now also U3.B18 (P1.12)
- net SDOUT: now also U3.B16 (P1.14)
- net SD_MODE: now also R33.2, R34.2, U3.AK16 (P0.20)
- net SWDCLK: now also J4.3 (Pin_3), U3.W31 (SWDCLK)
- net SWDIO: now also J4.2 (Pin_2), U3.AA31 (SWDIO)
- net TX: now also J3.1 (Pin_1)
- net VBUS: now also C26.2, J1.A4 (VBUS), J1.A9 (VBUS), J1.B4 (VBUS), J1.B9 (VBUS), R4.2, U4.B1 (VBUS), U4.B2 (VBUS)
- net VDD: now also R33.1, R34.1, C1.1, C10.2, C11.1, C12.1, C15.1, C27.2, C30.1, C31.1, C33.1, C34.1, C35.1, C36.1, C37.1, C38.1, C9.1, J4.1 (Pin_1), L5.1, LS1.5 (VDD), R10.2, R9.2, U1.10 (CSB), U1.3 (VDDIO), U1.7 (VDD), U2.20 (VDD), U3.A19 (VDD), U3.AC1 (VDD), U3.AG1 (VDD), U3.AJ31 (VDD), U3.AL11 (VDD), U3.AL17 (VDD), U3.AL25 (VDD), U3.AL3 (VDD), U3.AL7 (VDD), U3.B28 (VDD), U3.B8 (VDD), U3.C1 (VDD), U3.E1 (VDDH), U3.E31 (VDD), U3.L1 (VDD), U3.N31 (VDD), U3.U1 (VDD), U4.B5 (VOUTB), U4.C3 (VTERMSET)
- net VSYS: now also R11.2, R12.2, U4.C1 (VSYS), U4.C2 (VSYS); no longer R33.2, R34.2
- net nRESET: now also J4.5 (Pin_5), U3.AC31 (nRESET)
- new net: C13.1, C19.1, L3.1, U3.A27 (DECR), U3.G31 (DECRF)
- new net: R5.2, U4.E2 (ICHG)
- new net: C28.2, U4.A3 (DEC)
- new net: C14.1, R4.1, U3.A5 (VBUS)
- new net: U3.N1 (P0.00/XL1), Y2.2
- new net: U3.R1 (P0.01/XL2), Y2.1
- new net: C17.1, L4.1, U3.A15 (DECD)
- new net: L4.2, U3.B10 (DCCD)
- new net: C7.1, U3.B30 (XC2), Y1.2
- new net: C3.1, C4.1, L1.2, L2.1
- new net: R1.1, U2.7 (REXT)
- new net: AE1.1 (A), C5.1, L1.1
- new net: C20.1, U3.A13 (DECA)
- new net: L3.2, U3.A21 (DCCR)
- new net: L5.2, U4.A4 (SW)
- new net: J2.1 (Pin_1), U2.8 (ELE0)
- new net: J2.2 (Pin_2), U2.9 (ELE1)
- new net: J2.3 (Pin_3), U2.10 (ELE2)
- new net: C16.1, U3.B6 (DECUSB)
- new net: C8.1, U3.C31 (XC1), Y1.1
- new net: J1.B5 (CC2), R3.2
- new net: C2.1, U2.5 (VREG)
- new net: R6.2, U4.E1 (NTC)
- new net: D1.1 (K), U4.E3 (ERR)
- new net: D2.1 (K), U4.E4 (CHG)
- new net: D1.2 (A), R12.1
- new net: D2.2 (A), R11.1
- new net: C6.1, L2.2, U3.L31 (ANT)
- new net: J1.A5 (CC1), R2.2
- new net: C18.1, U3.A23 (DECN)
- no-connect marks 12 -> 22
Other:
- note added: "High-impedance input"
- note added: "Left"
- note added: "ON - MCU SD pin input (High impedance) OFF - MCU SD pin output (LOW)"
- note removed: "ISET LOW = 100mA USB limit ISET HIGH = 500mA USB limit"
- note removed: "Right"
- moved on the sheet: C22, C23, C24, C25, C29, C32, C42, C45, C49, C50, C51, J6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
