File: hardware/kicad/ver_1.0/MSBE_V3_BGA.kicad_pcb (KiCad board)
At the start: 2 copper layers, 82 parts, among them J1 High-V, J2 Low-V, J3 Low-V-TH, J4 Touch Pads, J5 UART, J6 USB, J7 Prog, U1 NPM1100-CAAA-R7, U3 MPR121QR2, U4 BMA400, U5 MAX98357AEWL_T

Commit message: pgrogress until decision to switch to 6-layer board
Parts:
- removed U5: MAX98357AEWL_T, mylib:MAX98357A_BGA9N40P3X3_134X143X69N
- added U2: NRF5340-CLAA-R, lib:NRF5340_CLAA_R, F.Cu at (119.9, 94.8)
- added U6: MAX98357AEWL_T, mylib:MAX98357A_BGA9N40P3X3_134X143X69N, F.Cu at (111.3, 96.3)
- added Y1: 32MHz, mylib:ECS-160-10-37-JTN-TR_ECS, F.Cu at (115.2, 91.9)
- added Y2: 32.768kHz, mylib:Pad_2Pin_1.5x0.8mm, F.Cu at (127.1, 95.0)
- J5, J6, J7: moved to B.Cu
- moved C1 96.6 mm to (54.8, 158.1)
- moved C10 96.6 mm to (57.7, 160.0)
- moved C2 96.6 mm to (54.8, 160.0)
- moved J1 96.6 mm to (54.7, 175.7)
- moved J2 96.6 mm to (57.2, 175.7)
- moved J3 96.6 mm to (70.0, 159.4)
- moved R1 96.6 mm to (73.8, 168.0)
- moved R4 96.6 mm to (76.7, 160.1)
- moved R5 96.6 mm to (76.7, 162.1)
- moved C11 96.6 mm to (57.7, 162.0)
- moved C6 96.6 mm to (54.8, 167.9)
- moved R10 96.6 mm to (79.6, 158.1)
- moved R13 96.6 mm to (79.6, 164.0)
- moved R14 96.6 mm to (79.6, 166.0)
- moved R2 96.6 mm to (73.8, 170.0)
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Connections:
- BT1 pad 3: (no net) -> GND
- C19 pad 1: +3.3V -> VDD
- C20 pad 1: +3.3V -> VDD
- C30 pad 2: +3.3V -> VDD
- C32 pad 1: +3.3V -> VDD
- C35 pad 1: +3.3V -> VDD
- C36 pad 2: +3.3V -> VDD
- C5 pad 2: +3.3V -> VDD
- J7 pad 1: +3.3V -> VDD
- L1 pad 1: +3.3V -> VDD
- LS1 pad 5: +3.3V -> VDD
- R15 pad 2: +3.3V -> VDD
- R16 pad 2: +3.3V -> VDD
- R20 pad 1: +3.3V -> VDD
- U1 pad B5: +3.3V -> VDD
- U1 pad C3: +3.3V -> VDD
- U3 pad 20: +3.3V -> VDD
- U4 pad 10: +3.3V -> VDD
- U4 pad 3: +3.3V -> VDD
- U4 pad 7: +3.3V -> VDD
Routing:
- net Net-(C24-Pad1): track 0.00 -> 20.9 mm, vias 0 -> 2
- net VDD: track 0.00 -> 13.0 mm, vias 0 -> 2
- net GND: track 0.00 -> 11.9 mm, vias 0 -> 2
- net /D-: track 0.00 -> 11.8 mm, vias 0 -> 2
- net /D+: track 0.00 -> 11.8 mm, vias 0 -> 2
- net Net-(U6-OUTP): track 0.00 -> 10.4 mm, vias 0 -> 2
- net +3.3V: track 0.00 -> 9.42 mm, vias 0 -> 1
- net /I2C_SDA: track 0.00 -> 8.48 mm, vias 0 -> 2
- net Net-(U2-DECR): track 0.00 -> 8.34 mm, vias 0 -> 3
- net VSYS: track 0.00 -> 8.24 mm, vias 0 -> 2
- net Net-(U6-OUTN): track 0.00 -> 7.87 mm
- net Net-(U2-P0.01/XL2): track 0.00 -> 6.98 mm, vias 0 -> 2
- net Net-(U2-VBUS): track 0.00 -> 6.79 mm, vias 0 -> 3
- net Net-(U2-XC2): track 0.00 -> 6.17 mm
- net /I2C_SCL: track 0.00 -> 5.45 mm, vias 0 -> 2
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- added copper zone on In1.Cu, net GND
Other:
- board outline added: 55.9 x 8.7 mm
- copper layers 2 -> 4
