File: hardware/kicad/ver_1.0/MSBE_V3_BGA.kicad_sch (KiCad schematic)
At the start: 90 parts, among them J1 USB_C_Receptacle_USB2.0_16P, J3 UART, J4 Prog, J5 Touch Pads, J6 High-V, J8 Low-V, J9 Low-V-TH, U1 NRF5340-CLAA-R, U3 NRF5340-QKAA-R, U4 NPM1100-CAAA-R7, U5 BMA400, U6 MAX98357AEWL_T, U7 MPR121QR2, Y1 32MHz, Y2 32.768kHz

Commit message: added version 4 BGA
Parts:
- removed C13: 1uF, Capacitor_SMD:C_0603_1608Metric, symbol Device:C
- removed C19: 2.2nF, Capacitor_SMD:C_0603_1608Metric, symbol Device:C
- removed C3, C4, C5: N.M., Capacitor_SMD:C_0603_1608Metric, symbol Device:C
- removed C35, C36, C37, C38: 100nF, Capacitor_SMD:C_0603_1608Metric, symbol Device:C
- removed C6: 0.7pF, Capacitor_SMD:C_0603_1608Metric, symbol Device:C
- removed J1: USB_C_Receptacle_USB2.0_16P, Connector_USB:USB_C_Receptacle_GCT_USB4110, symbol Connector:USB_C_Receptacle_USB2.0_16P
- removed J3: UART, myLib:Pad_3Pin_1.5x0.8mm, symbol Connector:Conn_01x03_Pin
- removed J4: Prog, myLib:Pad_prog_4Pad, symbol Connector:Conn_01x05_Pin
- removed L1: N.M., Inductor_SMD:L_0603_1608Metric, symbol Device:L
- removed R10, R9: 4k7, Resistor_SMD:R_0603_1608Metric, symbol Device:R
- removed R2, R3: 5K1R, Resistor_SMD:R_0603_1608Metric, symbol Device:R
- removed R4: 2R2, Resistor_SMD:R_0603_1608Metric, symbol Device:R
- removed U3: NRF5340-QKAA-R, myLib:NRF5340, symbol 1_MSBE_V3-altium-import:root_0_NRF5340-QKAA-R_
- added C21: 1uF, Capacitor_SMD:C_0402_1005Metric, symbol Device:C
- added C23, C24, C28: N.M., Capacitor_SMD:C_0402_1005Metric, symbol Device:C
- added C25, C27: 4.7uF, Capacitor_SMD:C_0402_1005Metric, symbol Device:C
- added C26: 100nF, Capacitor_SMD:C_0402_1005Metric, symbol Device:C
- added C29: 0.7pF, Capacitor_SMD:C_0402_1005Metric, symbol Device:C
- added J5: UART, mylib:Pad_3Pin_1.5x0.8mm, symbol Connector:Conn_01x03_Pin
- added J6: USB, mylib:Pad_4Pin_1.5x0.8mm, symbol Connector:Conn_01x04_Pin
- added J7: Prog, mylib:Pad_prog_4Pad, symbol Connector:Conn_01x05_Pin
- added L5: 2.2nH, Inductor_SMD:L_0402_1005Metric, symbol Device:L
- added R15, R16: 4.7k, Resistor_SMD:R_0402_1005Metric, symbol Device:R
- added R18: 2R2, Resistor_SMD:R_0402_1005Metric, symbol Device:R
- BT1: footprint myLib:Pad_3Pin_1.5x0.8mm -> mylib:Pad_3Pin_1.5x0.8mm
- C1: renamed from C42; footprint Capacitor_SMD:C_0603_1608Metric -> Capacitor_SMD:C_0402_1005Metric
- C10: renamed from C45; footprint Capacitor_SMD:C_0603_1608Metric -> Capacitor_SMD:C_0402_1005Metric
- C11: renamed from C51; footprint Capacitor_SMD:C_0603_1608Metric -> Capacitor_SMD:C_0402_1005Metric
- C12, C15, C18, C20, C31, C34, C8: footprint Capacitor_SMD:C_0603_1608Metric -> Capacitor_SMD:C_0402_1005Metric
- C13: renamed from C1; footprint Capacitor_SMD:C_0603_1608Metric -> Capacitor_SMD:C_0402_1005Metric
- C14: value 4.7uF -> 100nF; footprint Capacitor_SMD:C_0603_1608Metric -> Capacitor_SMD:C_0402_1005Metric
- C16: value 4.7uF -> 2.2nF; footprint Capacitor_SMD:C_0603_1608Metric -> Capacitor_SMD:C_0402_1005Metric
- C17: value 1uF -> 100nF; footprint Capacitor_SMD:C_0603_1608Metric -> Capacitor_SMD:C_0402_1005Metric
- C19: renamed from C29; footprint Capacitor_SMD:C_0603_1608Metric -> Capacitor_SMD:C_0402_1005Metric
- C2: renamed from C50; footprint Capacitor_SMD:C_0603_1608Metric -> Capacitor_SMD:C_0402_1005Metric
- C22: renamed from C39; footprint Capacitor_SMD:C_0603_1608Metric -> Capacitor_SMD:C_0402_1005Metric
- C3: renamed from C21; footprint Capacitor_SMD:C_0603_1608Metric -> Capacitor_SMD:C_0402_1005Metric
- C30: value 100nF -> 1uF; footprint Capacitor_SMD:C_0603_1608Metric -> Capacitor_SMD:C_0402_1005Metric
- C32: renamed from C9; footprint Capacitor_SMD:C_0603_1608Metric -> Capacitor_SMD:C_0402_1005Metric
- C33: value 100nF -> 0.1uF; footprint Capacitor_SMD:C_0603_1608Metric -> Capacitor_SMD:C_0402_1005Metric
- C35: renamed from C22; footprint Capacitor_SMD:C_0603_1608Metric -> Capacitor_SMD:C_0402_1005Metric
- C36: renamed from C24; footprint Capacitor_SMD:C_0603_1608Metric -> Capacitor_SMD:C_0402_1005Metric
- C37: renamed from C23; footprint Capacitor_SMD:C_0603_1608Metric -> Capacitor_SMD:C_0402_1005Metric
- C4: renamed from C26; footprint Capacitor_SMD:C_0603_1608Metric -> Capacitor_SMD:C_0402_1005Metric
- C5: renamed from C27; footprint Capacitor_SMD:C_0603_1608Metric -> Capacitor_SMD:C_0402_1005Metric
- C6: renamed from C49; footprint Capacitor_SMD:C_0603_1608Metric -> Capacitor_SMD:C_0402_1005Metric
- C7: renamed from C28; footprint Capacitor_SMD:C_0603_1608Metric -> Capacitor_SMD:C_0402_1005Metric
- C9: renamed from C7; footprint Capacitor_SMD:C_0603_1608Metric -> Capacitor_SMD:C_0402_1005Metric
- D1, D2: footprint LED_SMD:LED_0603_1608Metric -> LED_SMD:LED_0402_1005Metric
- J1: renamed from J6; footprint myLib:Pad_prog_4Pad -> mylib:Pad_4Pin_1.5x0.8mm
- J2: renamed from J8; footprint myLib:Pad_prog_4Pad -> mylib:Pad_4Pin_1.5x0.8mm
- J4: renamed from J5; footprint myLib:Pad_3Pin_1.5x0.8mm -> mylib:Pad_3Pin_1.5x0.8mm
- L1: renamed from L5; footprint Inductor_SMD:L_0603_1608Metric -> Inductor_SMD:L_0402_1005Metric
- L2: value 2.2nH -> 10uH; footprint Inductor_SMD:L_0603_1608Metric -> Inductor_SMD:L_0402_1005Metric
- L3: footprint Inductor_SMD:L_0603_1608Metric -> Inductor_SMD:L_0402_1005Metric
- L4: value 10uH -> N.M.; footprint Inductor_SMD:L_0603_1608Metric -> Inductor_SMD:L_0402_1005Metric
- LS1: footprint myLib:MIC_SPH18R1LM4H_KNO -> mylib:MIC_SPH18R1LM4H_KNO
- LS2: renamed from LS4; footprint myLib:Pad_2Pin_1.5x0.8mm -> mylib:Pad_2Pin_1.5x0.8mm
- LS3: renamed from LS5; footprint myLib:Pad_2Pin_1.5x0.8mm -> mylib:Pad_2Pin_1.5x0.8mm
- R1: renamed from R14; footprint Resistor_SMD:R_0603_1608Metric -> Resistor_SMD:R_0402_1005Metric
- R10: renamed from R23; footprint Resistor_SMD:R_0603_1608Metric -> Resistor_SMD:R_0402_1005Metric
- R11: renamed from R5; footprint Resistor_SMD:R_0603_1608Metric -> Resistor_SMD:R_0402_1005Metric
- R12: renamed from R6; footprint Resistor_SMD:R_0603_1608Metric -> Resistor_SMD:R_0402_1005Metric
- R13: renamed from R17; footprint Resistor_SMD:R_0603_1608Metric -> Resistor_SMD:R_0402_1005Metric
- R14: renamed from R25; footprint Resistor_SMD:R_0603_1608Metric -> Resistor_SMD:R_0402_1005Metric
- R17: renamed from R7; footprint Resistor_SMD:R_0603_1608Metric -> Resistor_SMD:R_0402_1005Metric
- R19: renamed from R8; footprint Resistor_SMD:R_0603_1608Metric -> Resistor_SMD:R_0402_1005Metric
- R2: renamed from R22; footprint Resistor_SMD:R_0603_1608Metric -> Resistor_SMD:R_0402_1005Metric
- R20: renamed from R34; footprint Resistor_SMD:R_0603_1608Metric -> Resistor_SMD:R_0402_1005Metric
- R3: renamed from R16; footprint Resistor_SMD:R_0603_1608Metric -> Resistor_SMD:R_0402_1005Metric
- R4: renamed from R24; footprint Resistor_SMD:R_0603_1608Metric -> Resistor_SMD:R_0402_1005Metric
- R5: renamed from R18; footprint Resistor_SMD:R_0603_1608Metric -> Resistor_SMD:R_0402_1005Metric
- R6: renamed from R19; footprint Resistor_SMD:R_0603_1608Metric -> Resistor_SMD:R_0402_1005Metric
- R7: renamed from R12; footprint Resistor_SMD:R_0603_1608Metric -> Resistor_SMD:R_0402_1005Metric
- R8: renamed from R11; footprint Resistor_SMD:R_0603_1608Metric -> Resistor_SMD:R_0402_1005Metric
- R9: renamed from R15; footprint Resistor_SMD:R_0603_1608Metric -> Resistor_SMD:R_0402_1005Metric
- U1: renamed from U4; footprint myLib:NPM1100-CAAA-BGA25C40P5X5_207X207X52N -> mylib:NPM1100-CAAA-BGA25C40P5X5_207X207X52N
- U3: renamed from U7; footprint myLib:MPR121 -> mylib:MPR121
- U4: renamed from U5; footprint myLib:QFN_BMA400_BOS -> mylib:QFN_BMA400_BOS
- U5: renamed from U6; footprint myLib:MAX98357A_BGA9N40P3X3_134X143X69N -> mylib:MAX98357A_BGA9N40P3X3_134X143X69N
- renumbered C25 to C38, C32 to C39, J9 to J3, U1 to U2
Connections:
- net +3.3V: now also C20.1, C30.2, U2.B10 (VDD), U2.B12 (VDDH), U2.B7 (VDD), U2.E11 (VDD), J7.1 (Pin_1), R15.2, R16.2; no longer C12.1, C15.1, C30.1, C31.1, C33.1, C34.1
- net AVSS: now also C12.1, C15.1, C16.1, C17.1, C30.1, U2.A5 (VSS), U2.B2 (VSS), U2.B9 (VSS), U2.C2 (VSS), U2.D12 (VSS), U2.E5 (VSS), U2.E6 (VSS), U2.E7 (VSS), U2.E8 (VSS), U2.F5 (VSS), U2.F6 (VSS), U2.F7 (VSS), U2.F8 (VSS), U2.G11 (P0.02/NFC1), U2.G6 (VSS), U2.G7 (VSS), U2.G8 (VSS), U2.H12 (P0.03/NFC2), U2.K6 (AVSS), C21.2, C23.2, C24.2, C25.1, C26.2, C27.1, C28.2, C29.2, J5.3 (Pin_3), J6.4 (Pin_4), J7.4 (Pin_4); no longer C12.2, C15.2, C16.2, C17.2, C30.2
- net D+: now also U2.A12 (D+), J6.2 (Pin_2)
- net D-: now also U2.A11 (D-), J6.3 (Pin_3)
- net I2C_SCL: now also U2.G10 (P0.04/AIN0), R15.1
- net I2C_SDA: now also U2.F10 (P0.05/AIN1), R16.1
- net INT1: now also U2.H10 (P0.06/AIN2)
- net INT2: now also U2.J10 (P0.07/AIN3)
- net IRQ: now also U2.J4 (P0.21)
- net ISET: now also U2.K4 (P0.22)
- net LRCLK: now also U2.C8 (P1.13)
- net MIC_CLOCK: now also U2.J2 (P0.26/AIN5)
- net MIC_DATA: now also U2.L1 (P0.25/AIN4)
- net RX: now also J5.2 (Pin_2)
- net SCK: now also U2.C7 (P1.12)
- net SDOUT: now also U2.C9 (P1.14)
- net SD_MODE: now also U2.K5 (P0.20)
- net SWDCLK: now also U2.F2 (SWDCLK), J7.3 (Pin_3)
- net SWDIO: now also U2.F1 (SWDIO), J7.2 (Pin_2)
- net TX: now also J5.1 (Pin_1)
- net VBUS: now also J6.1 (Pin_1), R18.2
- net nRESET: now also C33.1, U2.G2 (nRESET), J7.5 (Pin_5)
- net at L3.1: now also U2.B6 (DCC)
- net at C14.1: now also U2.A3 (VDD)
- net at Y2.2: now also U2.F11 (P0.00/XL1)
- net at Y2.1: now also U2.F12 (P0.01/XL2)
- net at L4.1: now also C24.1, C28.1, L5.1; no longer C17.1
- net at L4.2: now also AE1.1 (A), C23.1
- net at C9.1, Y1.2: now also U2.A1 (XC1)
- net at L2.1: now also U2.A9 (DCCD)
- net at L3.2: now also C15.2, C16.2, U2.B1 (DECRF), U2.B4 (DECR)
- net at C8.1, Y1.1: now also U2.A2 (XC2)
- net at L2.2: now also C12.2, U2.A7 (DECD)
- net at C18.1: now also U2.B5 (DECN)
- net at U2.B11 (VBUS): now also C27.2, R18.1
- net at U2.B8 (DECA): now also C21.1
- net at U2.C11 (DECUSB): now also C25.2
- net at U2.D1 (ANT): now also C29.1, L5.2
- net at U2.D2 (VDD): now also C26.1
- net at U2.H11 (VDD): now also C17.2
- net at U2.K1 (VDD): now also C34.1
- net at U2.L5 (VDD): now also C31.1
- no-connect marks 22 -> 10
Other:
- note added: "ISET_LOW = 100mA USB limit ISET_HIGH = 500mA USB limit"
- note removed: "Enable software pull-up"
- note removed: "High-impedance input"
- note removed: "Left"
- moved on the sheet: BT1, C1, C10, C11, C13, C19, C2, C22, C3, C32, C35, C36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

Commit message: pgrogress until decision to switch to 6-layer board
Parts:
- removed U5: MAX98357AEWL_T, mylib:MAX98357A_BGA9N40P3X3_134X143X69N, symbol lib:MAX98357AETE_
- added U6: MAX98357AEWL_T, mylib:MAX98357A_BGA9N40P3X3_134X143X69N, symbol lib:MAX98357AEWL_T
- U2: footprint WLCSP95_4.390X3.994_NOR -> lib:NRF5340_CLAA_R
- Y1: footprint myLib:ECS-160-10-37-JTN-TR_ECS -> mylib:ECS-160-10-37-JTN-TR_ECS
- Y2: footprint myLib:Crystal_24MHz-ECS-240-12-37B-CKY-TR -> mylib:Pad_2Pin_1.5x0.8mm
Connections:
- net +3.3V: now also U6.A2 (VDD); no longer C19.1, C20.1, C30.2, C32.1, C35.1, C36.2, C5.2, J7.1 (Pin_1), L1.1, LS1.5 (VDD), R15.2, R16.2, R20.1, U1.B5 (VOUTB), U1.C3 (VTERMSET), U2.B10 (VDD), U2.B12 (VDDH), U2.B7 (VDD), U2.E11 (VDD), U3.20 (VDD), U4.10 (CSB), U4.3 (VDDIO), U4.7 (VDD)
- net AVSS: now also U6.C2 (GND)
- net LRCLK: now also U6.B1 (DIN)
- net RX: now also U2.C10 (P1.15)
- net SCK: now also U6.C1 (BCLK)
- net SDOUT: now also U6.B2 (GAIN_SLOT)
- net SD_MODE: now also U6.A1 (SD_MODE)
- net TX: now also U2.E10 (P1.01)
- net at R19.2: now also U6.C3 (LRCLK)
- net at LS2.1, LS3.1: now also U6.B3 (OUTN)
- net at LS2.2, LS3.2: now also U6.A3 (OUTP)
- net at U1.A4 (SW): now also L1.1; no longer L1.2
- new net VDD: C19.1, C20.1, C30.2, C32.1, C35.1, C36.2, C5.2, J7.1 (Pin_1), L1.2, LS1.5 (VDD), R15.2, R16.2, R20.1, U1.B5 (VOUTB), U1.C3 (VTERMSET), U2.B10 (VDD), U2.B12 (VDDH), U2.B7 (VDD), U2.E11 (VDD), U3.20 (VDD), U4.10 (CSB), U4.3 (VDDIO), U4.7 (VDD)
Other:
- moved on the sheet: L1
