File: hardware/kicad/ver_1.0/MSBE_V3_BGA_6-layer.kicad_sch (KiCad schematic)
At the start: 67 parts, among them J4 Touch Pads, J5 UART, J6 USB, J7 Prog, U1 NPM1100-CAAA-R7, U2 NRF5340-CLAA-R, U3 MPR121QR2, U4 BMA400, U6 MAX98357AEWL_T, Y2 32.768kHz, Y3 32MHz

Commit message: continuing the idea of 6 layer board
Parts:
- added C1, C10, C11, C2, C6: 30pF, Capacitor_SMD:C_0402_1005Metric, symbol Device:C
- added J1: High-V, mylib:Pad_4Pin_1.5x0.8mm, symbol Connector:Conn_01x05_Pin
- added J2: Low-V, mylib:Pad_4Pin_1.5x0.8mm, symbol Connector:Conn_01x05_Pin
- added J3: Low-V-TH, Connector_PinHeader_2.54mm:PinHeader_1x05_P2.54mm_Vertical, symbol Connector:Conn_01x05_Pin
- added R1, R10, R2, R5, R9: 1K5, Resistor_SMD:R_0402_1005Metric, symbol Device:R
- added R13, R14, R3, R4, R6: 1K8, Resistor_SMD:R_0402_1005Metric, symbol Device:R
Connections:
- new net: R10.2, R14.2
- new net: R5.2, R6.2
- new net: R1.2, R3.2
- new net: R13.2, R9.2
- new net: R2.2, R4.2
- new net A1: C1.1, J1.1 (Pin_1), R1.1
- new net A2: C2.1, J1.2 (Pin_2), R2.1
- new net A3: C6.1, J1.3 (Pin_3), R5.1
- new net A4: C10.1, J1.4 (Pin_4), R9.1
- new net A5: C11.1, J1.5 (Pin_5), R10.1
- new net B1: C1.2, J2.1 (Pin_1), J3.5 (Pin_5), R3.1
- new net B2: C2.2, J2.2 (Pin_2), J3.4 (Pin_4), R4.1
- new net B3: C6.2, J2.3 (Pin_3), J3.3 (Pin_3), R6.1
- new net B4: C10.2, J2.4 (Pin_4), J3.2 (Pin_2), R13.1
- new net B5: C11.2, J2.5 (Pin_5), J3.1 (Pin_1), R14.1
Other:
- note added: "Logic Level Shifter Programing"
