File: hardware/kicad/ver_1.0/MSBE_V3_BGA_6-layer.kicad_pcb (KiCad board)
At the start: 4 copper layers, 55.9 x 8.7 mm, 67 parts, among them J4 Touch Pads, J5 UART, J6 USB, J7 Prog, U1 NPM1100-CAAA-R7, U2 NRF5340-CLAA-R, U3 MPR121QR2, U4 BMA400, U6 MAX98357AEWL_T, Y1 32MHz, Y2 32.768kHz

Commit message: continuing the idea of 6 layer board
Parts:
- added C1: 30pF, Capacitor_SMD:C_0402_1005Metric, F.Cu at (66.2, 141.1)
- added C10: 30pF, Capacitor_SMD:C_0402_1005Metric, F.Cu at (69.1, 143.1)
- added C11: 30pF, Capacitor_SMD:C_0402_1005Metric, F.Cu at (69.1, 145.1)
- added C2: 30pF, Capacitor_SMD:C_0402_1005Metric, F.Cu at (66.2, 143.1)
- added C6: 30pF, Capacitor_SMD:C_0402_1005Metric, F.Cu at (66.2, 151.0)
- added J1: High-V, mylib:Pad_4Pin_1.5x0.8mm, F.Cu at (66.1, 158.8)
- added J2: Low-V, mylib:Pad_4Pin_1.5x0.8mm, F.Cu at (68.6, 158.8)
- added J3: Low-V-TH, Connector_PinHeader_2.54mm:PinHeader_1x05_P2.54mm_Vertical, F.Cu at (81.4, 142.4)
- added R1: 1K5, Resistor_SMD:R_0402_1005Metric, F.Cu at (85.2, 151.1)
- added R10: 1K5, Resistor_SMD:R_0402_1005Metric, F.Cu at (91.0, 141.2)
- added R13: 1K8, Resistor_SMD:R_0402_1005Metric, F.Cu at (91.0, 147.1)
- added R14: 1K8, Resistor_SMD:R_0402_1005Metric, F.Cu at (91.0, 149.1)
- added R2: 1K5, Resistor_SMD:R_0402_1005Metric, F.Cu at (85.2, 153.1)
- added R3: 1K8, Resistor_SMD:R_0402_1005Metric, F.Cu at (88.1, 141.2)
- added R4: 1K8, Resistor_SMD:R_0402_1005Metric, F.Cu at (88.1, 143.1)
- added R5: 1K5, Resistor_SMD:R_0402_1005Metric, F.Cu at (88.1, 145.1)
- added R6: 1K8, Resistor_SMD:R_0402_1005Metric, F.Cu at (88.1, 147.1)
- added R9: 1K5, Resistor_SMD:R_0402_1005Metric, F.Cu at (88.1, 153.1)
Routing:
- net +3.3V: track 0.00 -> 12.1 mm, vias 0 -> 1
- net GND: track 0.00 -> 10.2 mm
- net Net-(U2-DECR): track 0.00 -> 8.99 mm, vias 0 -> 3
- net Net-(U2-XC2): track 0.00 -> 6.17 mm
- net Net-(U2-DECN): track 0.00 -> 5.02 mm, vias 0 -> 2
- net Net-(U2-DECA): track 0.00 -> 4.25 mm, vias 0 -> 2
- net Net-(U2-XC1): track 0.00 -> 3.63 mm
- net Net-(U2-DECD): track 0.00 -> 2.97 mm, vias 0 -> 2
- net Net-(U2-DCC): track 0.00 -> 2.92 mm, vias 0 -> 2
- net Net-(U2-DCCD): track 0.00 -> 2.38 mm, vias 0 -> 2
- net Net-(C14-Pad1): track 0.00 -> 1.44 mm
- net VDD: track 0.00 -> 0.97 mm
- added copper zone on In1.Cu, net GND
Other:
- copper layers 4 -> 6

Commit message: added test for Claude + KiCad
Parts:
- turned Y2 to -90 degrees
Routing:
- net Net-(C24-Pad1): track 0.00 -> 19.3 mm, vias 0 -> 2
- net /D+: track 0.00 -> 10.6 mm, vias 0 -> 2
- net /D-: track 0.00 -> 10.6 mm, vias 0 -> 2
- net Net-(U2-P0.00/XL1): track 0.00 -> 6.86 mm, vias 0 -> 2
- net /I2C_SDA: track 0.00 -> 6.34 mm, vias 0 -> 2
- net Net-(C26-Pad1): track 0.00 -> 5.97 mm, vias 0 -> 2
- net Net-(U2-VBUS): track 0.00 -> 5.91 mm, vias 0 -> 3
- net /I2C_SCL: track 0.00 -> 5.14 mm, vias 0 -> 2
- net Net-(U2-P0.01/XL2): track 0.00 -> 4.06 mm
- net Net-(U2-ANT): track 0.00 -> 3.52 mm
- net /nRESET: track 0.00 -> 3.26 mm
- net GND: track 10.2 -> 13.2 mm
- net Net-(C34-Pad1): track 0.00 -> 2.42 mm
- net Net-(C17-Pad2): track 0.00 -> 2.37 mm, vias 0 -> 2
- net Net-(U2-DECUSB): track 0.00 -> 2.32 mm
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