File: hardware/kicad/ver_1.0 - test/MSBE_V3_BGA_6-layer.kicad_pcb (KiCad board)
At the start: 6 copper layers, 55.9 x 8.7 mm, 85 parts, among them J1 High-V, J2 Low-V, J3 Low-V-TH, J4 Touch Pads, J5 UART, J6 USB, J7 Prog, U1 NPM1100-CAAA-R7, U2 NRF5340-CLAA-R, U3 MPR121QR2, U4 BMA400, U6 MAX98357AEWL_T, Y2 32.768kHz, Y3 32MHz

Commit message: added silckscreen
Parts:
- added H-IN: High-V-TH, Connector_PinHeader_2.54mm:PinHeader_1x05_P2.54mm_Vertical, F.Cu at (89.4, 114.1)
- added REF**: Pad_3Pin_1.5x0.8mm, mylib:Pad_3Pin_1.5x0.8mm, B.Cu at (133.5, 103.2)
- J1, J2: footprint mylib:Pad_4Pin_1.5x0.8mm -> mylib:Pad_prog_4Pad
- moved R9 48.2 mm to (98.0, 105.5)
- moved R14 48.1 mm to (98.0, 104.0)
- moved R13 44.6 mm to (98.0, 106.8)
- moved R10 43.2 mm to (98.0, 102.8)
- moved R2 41.9 mm to (98.0, 111.1)
- moved J1 41.9 mm to (93.2, 109.6)
- moved J2 40.7 mm to (101.6, 109.6)
- moved R6 40.6 mm to (98.0, 109.5)
- moved R5 40.1 mm to (98.0, 108.2)
- moved R1 38.5 mm to (98.0, 113.7)
- moved R4 36.1 mm to (98.0, 112.4)
- moved C11 34.7 mm to (96.5, 103.4), turned to -90 degrees
- moved C6 34.3 mm to (96.5, 108.8), turned to -90 degrees
- moved R3 33.5 mm to (98.0, 114.9)
- moved L-OUT 33.3 mm to (104.9, 103.9)
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- renumbered J3 to L-OUT
Routing:
- net /B1: track 0.00 -> 12.4 mm
- net /B2: track 0.00 -> 11.0 mm
- net /A5: track 0.00 -> 10.9 mm
- net /B5: track 0.00 -> 10.6 mm
- net /A1: track 0.00 -> 10.2 mm
- net /A4: track 0.00 -> 9.58 mm
- net /B4: track 0.00 -> 9.46 mm
- net /B3: track 0.00 -> 9.20 mm
- net /A2: track 0.00 -> 9.13 mm
- net /A3: track 0.00 -> 8.46 mm
- net Net-(J4-Pin_1): track 4.49 -> 10.4 mm, vias 2 -> 3
- net Net-(J4-Pin_3): track 1.43 -> 4.46 mm, vias 0 -> 1
- net Net-(R2-Pad2): track 0.00 -> 1.27 mm
- net Net-(R10-Pad2): track 0.00 -> 1.27 mm
- net Net-(R5-Pad2): track 0.00 -> 1.26 mm
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- added copper zone on F.Cu, net Net-(J4-Pin_1)
- added copper zone on F.Cu, net Net-(J4-Pin_2)
- added copper zone on F.Cu, net Net-(J4-Pin_3)
Other:
- board size 55.9 x 8.7 mm -> 55.9 x 25.5 mm
- board text added: "*"
- board text added: "+"
- board text added: "-"
- board text added: "-->"
- board text added: "1K5"
- board text added: "High to Low V-Convertor"
- board text added: "MSBE 0100 1101"
- board text added: "PROG"
- board text added: "RIGHT LEFT"
- board text added: "Touch sensor"
- board text added: "UART"
- board text added: "USB"
